File: hardware/8x8/led_4x2_left.kicad_sch (KiCad schematic)
At the start: 20 parts

Commit message: Completed Major Routing
Parts:
- removed LD? (x8): WP154A4SEJ3VBDZGC/CA, RGB LED:WP154A4SEJ3VBDZGC&slash_CA, symbol RGB LED:WP154A4SEJ3VBDZGC{brace}slash}CA
- added LD1, LD2, LD3, LD4, LD5, LD6, LD7, LD8: WP154A4SEJ3VBDZGC/CA, RGB LED:WP154A4SEJ3VBDZGC&slash_CA, symbol RGB LED:WP154A4SEJ3VBDZGC{brace}slash}CA
Connections:
- net +5V: now also LD1.2 (CA), LD2.2 (CA), LD3.2 (CA), LD4.2 (CA), LD5.2 (CA), LD6.2 (CA), LD7.2 (CA), LD8.2 (CA)
- net LD1_B: now also DRV1.19 (LED11), LD1.3 (B); no longer DRV1.6 (LED0)
- net LD1_G: now also DRV1.17 (LED10), LD1.4 (G); no longer DRV1.7 (LED1)
- net LD1_R: now also LD1.1 (R)
- net LD2_B: now also DRV1.16 (LED9), LD2.3 (B); no longer DRV1.8 (LED2)
- net LD2_G: now also DRV1.15 (LED8), LD2.4 (G); no longer DRV1.9 (LED3)
- net LD2_R: now also LD2.1 (R)
- net LD3_B: now also DRV1.13 (LED7), LD3.3 (B); no longer DRV1.10 (LED4)
- net LD3_G: now also DRV1.12 (LED6), LD3.4 (G); no longer DRV1.11 (LED5)
- net LD3_R: now also LD3.1 (R)
- net LD4_B: now also DRV1.11 (LED5), LD4.3 (B); no longer DRV1.12 (LED6)
- net LD4_G: now also DRV1.10 (LED4), LD4.4 (G); no longer DRV1.13 (LED7)
- net LD4_R: now also LD4.1 (R)
- net LD5_B: now also DRV1.20 (LED12), LD5.3 (B); no longer DRV1.33 (LED23)
- net LD5_G: now also DRV1.22 (LED13), LD5.4 (G); no longer DRV1.32 (LED22)
- net LD5_R: now also LD5.1 (R)
- net LD6_B: now also DRV1.23 (LED14), LD6.3 (B); no longer DRV1.31 (LED21)
- net LD6_G: now also DRV1.24 (LED15), LD6.4 (G); no longer DRV1.30 (LED20)
- net LD6_R: now also LD6.1 (R)
- net LD7_B: now also DRV1.26 (LED16), LD7.3 (B); no longer DRV1.29 (LED19)
- net LD7_G: now also DRV1.27 (LED17), LD7.4 (G); no longer DRV1.28 (LED18)
- net LD7_R: now also LD7.1 (R)
- net LD8_B: now also DRV1.28 (LED18), LD8.3 (B); no longer DRV1.27 (LED17)
- net LD8_G: now also DRV1.29 (LED19), LD8.4 (G); no longer DRV1.26 (LED16)
- net LD8_R: now also LD8.1 (R)
- net SR1_R: now also DRV1.6 (LED0); no longer DRV1.19 (LED11)
- net SR2_R: now also DRV1.7 (LED1); no longer DRV1.17 (LED10)
- net SR3_R: now also DRV1.8 (LED2); no longer DRV1.16 (LED9)
- net SR4_R: now also DRV1.9 (LED3); no longer DRV1.15 (LED8)
- net SR5_R: now also DRV1.33 (LED23); no longer DRV1.24 (LED15)
- net SR6_R: now also DRV1.32 (LED22); no longer DRV1.23 (LED14)
- net SR7_R: now also DRV1.31 (LED21); no longer DRV1.22 (LED13)
- net SR8_R: now also DRV1.30 (LED20); no longer DRV1.20 (LED12)
- net  LDRow_Amps/Amp_IP_1 renamed  LDRow_Amps1/Amp_IP_2
- net  LDRow_Amps/Amp_IP_2 renamed  LDRow_Amps1/Amp_IP_1
- net  LDRow_Amps/Amp_IP_3 renamed  LDRow_Amps1/Amp_IP_4
- net  LDRow_Amps/Amp_IP_4 renamed  LDRow_Amps1/Amp_IP_3
- net  LDRow_Amps/Amp_IP_5 renamed  LDRow_Amps1/Amp_IP_6
- net  LDRow_Amps/Amp_IP_6 renamed  LDRow_Amps1/Amp_IP_5
- net  LDRow_Amps/Amp_IP_7 renamed  LDRow_Amps1/Amp_IP_8
- net  LDRow_Amps/Amp_IP_8 renamed  LDRow_Amps1/Amp_IP_7
- net  LDRow_Amps/Amp_OP_1 renamed  LDRow_Amps1/Amp_OP_5
- net  LDRow_Amps/Amp_OP_2 renamed  LDRow_Amps1/Amp_OP_6
- net  LDRow_Amps/Amp_OP_3 renamed  LDRow_Amps1/Amp_OP_7
- net  LDRow_Amps/Amp_OP_4 renamed  LDRow_Amps1/Amp_OP_8
- net  LDRow_Amps/Amp_OP_5 renamed  LDRow_Amps1/Amp_OP_1
- net  LDRow_Amps/Amp_OP_6 renamed  LDRow_Amps1/Amp_OP_2
- net  LDRow_Amps/Amp_OP_7 renamed  LDRow_Amps1/Amp_OP_3
- net  LDRow_Amps/Amp_OP_8 renamed  LDRow_Amps1/Amp_OP_4
Other:
- removed sheet  LDRow_Amps
- added sheet  LDRow_Amps1 (led_row_amps.kicad_sch)
