File: hardware/8x8/led_4x2_right.kicad_sch (KiCad schematic)
At the start: 20 parts

Commit message: Completed Major Routing
Parts:
- removed AD1: MCU-MCP3008-I/P(DIP16-7.62MM), ADC:MCP3008-I&slash_P, symbol ADC:MCU-MCP3008-I{brace}slash}P(DIP16-7.62MM)
- removed DRV1: PCA9956BTWY, LED Driver:SOP50P640X110-39N, symbol LED Driver:PCA9956BTWY
- removed ISEL1: 2K, Resistor TH:footprints, symbol Device:R
- removed LD? (x8): WP154A4SEJ3VBDZGC/CA, RGB LED:WP154A4SEJ3VBDZGC&slash_CA, symbol RGB LED:WP154A4SEJ3VBDZGC{brace}slash}CA
- removed PU1: 10K, Resistor TH:footprints, symbol Device:R
- removed SR1, SR2, SR3, SR4, SR5, SR6, SR7, SR8: TLP4176ATP_F, SSR:footprints, symbol SSR:TLP4176ATP_F
- added AD2: MCU-MCP3008-I/P(DIP16-7.62MM), ADC:MCP3008-I&slash_P, symbol ADC:MCU-MCP3008-I{brace}slash}P(DIP16-7.62MM)
- added DRV2: PCA9956BTWY, LED Driver:SOP50P640X110-39N, symbol LED Driver:PCA9956BTWY
- added ISEL2: 2K, Resistor TH:footprints, symbol Device:R
- added LD10, LD11, LD12, LD13, LD14, LD15, LD16, LD9: WP154A4SEJ3VBDZGC/CA, RGB LED:WP154A4SEJ3VBDZGC&slash_CA, symbol RGB LED:WP154A4SEJ3VBDZGC{brace}slash}CA
- added PU2: 10K, Resistor TH:footprints, symbol Device:R
- added SR10, SR11, SR12, SR13, SR14, SR15, SR16, SR9: TLP4176ATP_F, SSR:footprints, symbol SSR:TLP4176ATP_F
Connections:
- net  LDRow_Amps/Amp_IP_1: now also SR9.3 (Load)
- net  LDRow_Amps/Amp_IP_2: now also SR10.3 (Load)
- net  LDRow_Amps/Amp_IP_3: now also SR14.3 (Load)
- net  LDRow_Amps/Amp_IP_4: now also SR13.3 (Load)
- net  LDRow_Amps/Amp_IP_5: now also SR11.3 (Load)
- net  LDRow_Amps/Amp_IP_6: now also SR12.3 (Load)
- net  LDRow_Amps/Amp_IP_7: now also SR16.3 (Load)
- net  LDRow_Amps/Amp_IP_8: now also SR15.3 (Load)
- net  LDRow_Amps/Amp_OP_1: now also AD2.8 (CH7)
- net  LDRow_Amps/Amp_OP_2: now also AD2.7 (CH6)
- net  LDRow_Amps/Amp_OP_3: now also AD2.2 (CH1)
- net  LDRow_Amps/Amp_OP_4: now also AD2.1 (CH0)
- net  LDRow_Amps/Amp_OP_5: now also AD2.6 (CH5)
- net  LDRow_Amps/Amp_OP_6: now also AD2.5 (CH4)
- net  LDRow_Amps/Amp_OP_7: now also AD2.4 (CH3)
- net  LDRow_Amps/Amp_OP_8: now also AD2.3 (CH2)
- net +5V: now also AD2.15 (VREF), AD2.16 (VDD), DRV2.38 (VDD), LD10.2 (CA), LD11.2 (CA), LD12.2 (CA), LD13.2 (CA), LD14.2 (CA), LD15.2 (CA), LD16.2 (CA), LD9.2 (CA), PU2.1
- net ADC_SHDN: now also AD2.10 (SHDN/~{CS})
- net Drv_AD0: now also DRV2.2 (AD0)
- net Drv_AD1: now also DRV2.3 (AD1)
- net GND: now also AD2.14 (AGND), AD2.9 (DGND), DRV2.14 (VSS), DRV2.18 (VSS), DRV2.21 (VSS), DRV2.25 (VSS), DRV2.34 (VSS), DRV2.39 (EXP), DRV2.4 (AD2), DRV2.5 (~{OE}), ISEL2.1
- net I2C_SCL: now also DRV2.36 (SCL)
- net I2C_SDA_5V: now also DRV2.37 (SDA)
- net LD1_B: now also DRV2.13 (LED7), LD9.3 (B)
- net LD1_G: now also DRV2.12 (LED6), LD9.4 (G)
- net LD1_R: now also LD9.1 (R), SR9.1 (+Ctr), SR9.4 (Load)
- net LD2_B: now also DRV2.11 (LED5), LD10.3 (B)
- net LD2_G: now also DRV2.10 (LED4), LD10.4 (G)
- net LD2_R: now also LD10.1 (R), SR10.1 (+Ctr), SR10.4 (Load)
- net LD3_B: now also DRV2.9 (LED3), LD11.3 (B)
- net LD3_G: now also DRV2.8 (LED2), LD11.4 (G)
- net LD3_R: now also LD11.1 (R), SR11.1 (+Ctr), SR11.4 (Load)
- net LD4_B: now also DRV2.7 (LED1), LD12.3 (B)
- net LD4_G: now also DRV2.6 (LED0), LD12.4 (G)
- net LD4_R: now also LD12.1 (R), SR12.1 (+Ctr), SR12.4 (Load)
- net LD5_B: now also DRV2.26 (LED16), LD13.3 (B)
- net LD5_G: now also DRV2.27 (LED17), LD13.4 (G)
- net LD5_R: now also LD13.1 (R), SR13.1 (+Ctr), SR13.4 (Load)
- net LD6_B: now also DRV2.28 (LED18), LD14.3 (B)
- net LD6_G: now also DRV2.29 (LED19), LD14.4 (G)
- net LD6_R: now also LD14.1 (R), SR14.1 (+Ctr), SR14.4 (Load)
- net LD7_B: now also DRV2.30 (LED20), LD15.3 (B)
- net LD7_G: now also DRV2.31 (LED21), LD15.4 (G)
- net LD7_R: now also LD15.1 (R), SR15.1 (+Ctr), SR15.4 (Load)
- net LD8_B: now also DRV2.32 (LED22), LD16.3 (B)
- net LD8_G: now also DRV2.33 (LED23), LD16.4 (G)
- net LD8_R: now also LD16.1 (R), SR16.1 (+Ctr), SR16.4 (Load)
- net SPI_MISO_5V: now also AD2.12 (DOUT)
- net SPI_MOSI: now also AD2.11 (DIN)
- net SPI_SCK: now also AD2.13 (CLK)
- net SR1_R: now also DRV2.15 (LED8), SR9.2 (-Ctr)
- net SR2_R: now also DRV2.16 (LED9), SR10.2 (-Ctr)
- net SR3_R: now also DRV2.17 (LED10), SR11.2 (-Ctr)
- net SR4_R: now also DRV2.19 (LED11), SR12.2 (-Ctr)
- net SR5_R: now also DRV2.24 (LED15), SR13.2 (-Ctr)
- net SR6_R: now also DRV2.23 (LED14), SR14.2 (-Ctr)
- net SR7_R: now also DRV2.22 (LED13), SR15.2 (-Ctr)
- net SR8_R: now also DRV2.20 (LED12), SR16.2 (-Ctr)
- new net: DRV2.1 (REXT), ISEL2.2
- new net: DRV2.35 (~{RESET}), PU2.2
