File: hardware/8x8/8x8.kicad_pcb (KiCad board)
At the start: 2 copper layers, 0 parts

Commit message: Temporary Component Placement on PCB
Parts:
- added ADC_1: MCP3008-I/P-DIP16, ADC:MCP3008-I&slash_P, F.Cu at (182.9, 53.3)
- added ADC_2: MCP3008-I/P-DIP16, ADC:MCP3008-I&slash_P, F.Cu at (182.9, 66.0)
- added ADC_3: MCP3008-I/P-DIP16, ADC:MCP3008-I&slash_P, F.Cu at (182.9, 78.7)
- added ADC_4: MCP3008-I/P-DIP16, ADC:MCP3008-I&slash_P, F.Cu at (182.9, 91.4)
- added ADC_5: MCP3008-I/P-DIP16, ADC:MCP3008-I&slash_P, F.Cu at (182.9, 104.1)
- added ADC_6: MCP3008-I/P-DIP16, ADC:MCP3008-I&slash_P, F.Cu at (182.9, 116.8)
- added ADC_7: MCP3008-I/P-DIP16, ADC:MCP3008-I&slash_P, F.Cu at (182.9, 129.5)
- added ADC_8: MCP3008-I/P-DIP16, ADC:MCP3008-I&slash_P, F.Cu at (182.9, 142.2)
- added AMP_1: MCP619-I/SL, Op-Amp:footprints, F.Cu at (203.2, 53.3)
- added AMP_10: MCP619-I/SL, Op-Amp:footprints, F.Cu at (238.8, 104.1)
- added AMP_11: MCP619-I/SL, Op-Amp:footprints, F.Cu at (203.2, 116.8)
- added AMP_12: MCP619-I/SL, Op-Amp:footprints, F.Cu at (238.8, 116.8)
- added AMP_13: MCP619-I/SL, Op-Amp:footprints, F.Cu at (203.2, 129.5)
- added AMP_14: MCP619-I/SL, Op-Amp:footprints, F.Cu at (238.8, 129.5)
- added AMP_15: MCP619-I/SL, Op-Amp:footprints, F.Cu at (203.2, 142.2)
- added AMP_16: MCP619-I/SL, Op-Amp:footprints, F.Cu at (238.8, 142.2)
- added AMP_2: MCP619-I/SL, Op-Amp:footprints, F.Cu at (238.8, 53.3)
- added AMP_3: MCP619-I/SL, Op-Amp:footprints, F.Cu at (203.2, 66.1)
- added AMP_4: MCP619-I/SL, Op-Amp:footprints, F.Cu at (238.8, 66.1)
- added AMP_5: MCP619-I/SL, Op-Amp:footprints, F.Cu at (203.2, 78.7)
- added AMP_6: MCP619-I/SL, Op-Amp:footprints, F.Cu at (238.8, 78.7)
- added AMP_7: MCP619-I/SL, Op-Amp:footprints, F.Cu at (203.2, 91.4)
- added AMP_8: MCP619-I/SL, Op-Amp:footprints, F.Cu at (238.8, 91.4)
- added AMP_9: MCP619-I/SL, Op-Amp:footprints, F.Cu at (203.2, 104.1)
- added Addr_Sel_1: 100K, Resistor_THT:R_Axial_DIN0207_L6.3mm_D2.5mm_P7.62mm_Horizontal, F.Cu at (295.9, 50.8)
- added Addr_Sel_2: 100K, Resistor_THT:R_Axial_DIN0207_L6.3mm_D2.5mm_P7.62mm_Horizontal, F.Cu at (295.9, 63.5)
- added Addr_Sel_3: 100K, Resistor_THT:R_Axial_DIN0207_L6.3mm_D2.5mm_P7.62mm_Horizontal, F.Cu at (295.9, 68.6)
- added Addr_Sel_4: 100K, Resistor_THT:R_Axial_DIN0207_L6.3mm_D2.5mm_P7.62mm_Horizontal, F.Cu at (295.9, 76.2)
- added Addr_Sel_5: 100K, Resistor_THT:R_Axial_DIN0207_L6.3mm_D2.5mm_P7.62mm_Horizontal, F.Cu at (295.9, 106.7)
- added Addr_Sel_6: 100K, Resistor_THT:R_Axial_DIN0207_L6.3mm_D2.5mm_P7.62mm_Horizontal, F.Cu at (295.9, 132.1)
- added Amp_Fdbk_1: 2M, Resistor_THT:R_Axial_DIN0207_L6.3mm_D2.5mm_P7.62mm_Horizontal, F.Cu at (210.8, 50.8)
- added Amp_Fdbk_10: 2M, Resistor_THT:R_Axial_DIN0207_L6.3mm_D2.5mm_P7.62mm_Horizontal, F.Cu at (210.9, 68.6)
- added Amp_Fdbk_11: 2M, Resistor_THT:R_Axial_DIN0207_L6.3mm_D2.5mm_P7.62mm_Horizontal, F.Cu at (222.2, 63.5)
- added Amp_Fdbk_12: 2M, Resistor_THT:R_Axial_DIN0207_L6.3mm_D2.5mm_P7.62mm_Horizontal, F.Cu at (222.2, 68.6)
- added Amp_Fdbk_13: 2M, Resistor_THT:R_Axial_DIN0207_L6.3mm_D2.5mm_P7.62mm_Horizontal, F.Cu at (246.4, 63.5)
- added Amp_Fdbk_14: 2M, Resistor_THT:R_Axial_DIN0207_L6.3mm_D2.5mm_P7.62mm_Horizontal, F.Cu at (246.4, 68.6)
- added Amp_Fdbk_15: 2M, Resistor_THT:R_Axial_DIN0207_L6.3mm_D2.5mm_P7.62mm_Horizontal, F.Cu at (257.8, 63.5)
- added Amp_Fdbk_16: 2M, Resistor_THT:R_Axial_DIN0207_L6.3mm_D2.5mm_P7.62mm_Horizontal, F.Cu at (257.8, 68.6)
- added Amp_Fdbk_17: 2M, Resistor_THT:R_Axial_DIN0207_L6.3mm_D2.5mm_P7.62mm_Horizontal, F.Cu at (210.9, 76.2)
- added Amp_Fdbk_18: 2M, Resistor_THT:R_Axial_DIN0207_L6.3mm_D2.5mm_P7.62mm_Horizontal, F.Cu at (210.9, 81.3)
- added Amp_Fdbk_19: 2M, Resistor_THT:R_Axial_DIN0207_L6.3mm_D2.5mm_P7.62mm_Horizontal, F.Cu at (222.2, 76.2)
- added Amp_Fdbk_2: 2M, Resistor_THT:R_Axial_DIN0207_L6.3mm_D2.5mm_P7.62mm_Horizontal, F.Cu at (210.9, 55.9)
- added Amp_Fdbk_20: 2M, Resistor_THT:R_Axial_DIN0207_L6.3mm_D2.5mm_P7.62mm_Horizontal, F.Cu at (222.2, 81.3)
- added Amp_Fdbk_21: 2M, Resistor_THT:R_Axial_DIN0207_L6.3mm_D2.5mm_P7.62mm_Horizontal, F.Cu at (246.4, 76.2)
- added Amp_Fdbk_22: 2M, Resistor_THT:R_Axial_DIN0207_L6.3mm_D2.5mm_P7.62mm_Horizontal, F.Cu at (246.4, 81.3)
- added Amp_Fdbk_23: 2M, Resistor_THT:R_Axial_DIN0207_L6.3mm_D2.5mm_P7.62mm_Horizontal, F.Cu at (257.8, 76.2)
- added Amp_Fdbk_24: 2M, Resistor_THT:R_Axial_DIN0207_L6.3mm_D2.5mm_P7.62mm_Horizontal, F.Cu at (257.8, 81.3)
- added Amp_Fdbk_25: 2M, Resistor_THT:R_Axial_DIN0207_L6.3mm_D2.5mm_P7.62mm_Horizontal, F.Cu at (210.8, 88.9)
- added Amp_Fdbk_26: 2M, Resistor_THT:R_Axial_DIN0207_L6.3mm_D2.5mm_P7.62mm_Horizontal, F.Cu at (210.8, 94.0)
- added Amp_Fdbk_27: 2M, Resistor_THT:R_Axial_DIN0207_L6.3mm_D2.5mm_P7.62mm_Horizontal, F.Cu at (222.2, 88.9)
- added Amp_Fdbk_28: 2M, Resistor_THT:R_Axial_DIN0207_L6.3mm_D2.5mm_P7.62mm_Horizontal, F.Cu at (222.2, 94.0)
- added Amp_Fdbk_29: 2M, Resistor_THT:R_Axial_DIN0207_L6.3mm_D2.5mm_P7.62mm_Horizontal, F.Cu at (246.4, 88.9)
- added Amp_Fdbk_3: 2M, Resistor_THT:R_Axial_DIN0207_L6.3mm_D2.5mm_P7.62mm_Horizontal, F.Cu at (222.2, 50.8)
- added Amp_Fdbk_30: 2M, Resistor_THT:R_Axial_DIN0207_L6.3mm_D2.5mm_P7.62mm_Horizontal, F.Cu at (246.4, 94.0)
- added Amp_Fdbk_31: 2M, Resistor_THT:R_Axial_DIN0207_L6.3mm_D2.5mm_P7.62mm_Horizontal, F.Cu at (257.8, 88.9)
- added Amp_Fdbk_32: 2M, Resistor_THT:R_Axial_DIN0207_L6.3mm_D2.5mm_P7.62mm_Horizontal, F.Cu at (257.8, 94.0)
- added Amp_Fdbk_33: 2M, Resistor_THT:R_Axial_DIN0207_L6.3mm_D2.5mm_P7.62mm_Horizontal, F.Cu at (210.8, 101.6)
- added Amp_Fdbk_34: 2M, Resistor_THT:R_Axial_DIN0207_L6.3mm_D2.5mm_P7.62mm_Horizontal, F.Cu at (210.8, 106.7)
- added Amp_Fdbk_35: 2M, Resistor_THT:R_Axial_DIN0207_L6.3mm_D2.5mm_P7.62mm_Horizontal, F.Cu at (222.2, 101.6)
- added Amp_Fdbk_36: 2M, Resistor_THT:R_Axial_DIN0207_L6.3mm_D2.5mm_P7.62mm_Horizontal, F.Cu at (222.2, 106.7)
- added Amp_Fdbk_37: 2M, Resistor_THT:R_Axial_DIN0207_L6.3mm_D2.5mm_P7.62mm_Horizontal, F.Cu at (246.4, 101.6)
- added Amp_Fdbk_38: 2M, Resistor_THT:R_Axial_DIN0207_L6.3mm_D2.5mm_P7.62mm_Horizontal, F.Cu at (246.4, 106.7)
- added Amp_Fdbk_39: 2M, Resistor_THT:R_Axial_DIN0207_L6.3mm_D2.5mm_P7.62mm_Horizontal, F.Cu at (257.8, 101.6)
- added Amp_Fdbk_4: 2M, Resistor_THT:R_Axial_DIN0207_L6.3mm_D2.5mm_P7.62mm_Horizontal, F.Cu at (222.2, 55.9)
- added Amp_Fdbk_40: 2M, Resistor_THT:R_Axial_DIN0207_L6.3mm_D2.5mm_P7.62mm_Horizontal, F.Cu at (257.8, 106.7)
- added Amp_Fdbk_41: 2M, Resistor_THT:R_Axial_DIN0207_L6.3mm_D2.5mm_P7.62mm_Horizontal, F.Cu at (210.8, 114.3)
- added Amp_Fdbk_42: 2M, Resistor_THT:R_Axial_DIN0207_L6.3mm_D2.5mm_P7.62mm_Horizontal, F.Cu at (210.8, 119.4)
- added Amp_Fdbk_43: 2M, Resistor_THT:R_Axial_DIN0207_L6.3mm_D2.5mm_P7.62mm_Horizontal, F.Cu at (222.2, 114.3)
- added Amp_Fdbk_44: 2M, Resistor_THT:R_Axial_DIN0207_L6.3mm_D2.5mm_P7.62mm_Horizontal, F.Cu at (222.2, 119.4)
- added Amp_Fdbk_45: 2M, Resistor_THT:R_Axial_DIN0207_L6.3mm_D2.5mm_P7.62mm_Horizontal, F.Cu at (246.4, 114.3)
- added Amp_Fdbk_46: 2M, Resistor_THT:R_Axial_DIN0207_L6.3mm_D2.5mm_P7.62mm_Horizontal, F.Cu at (246.4, 119.4)
- added Amp_Fdbk_47: 2M, Resistor_THT:R_Axial_DIN0207_L6.3mm_D2.5mm_P7.62mm_Horizontal, F.Cu at (257.8, 114.3)
- added Amp_Fdbk_48: 2M, Resistor_THT:R_Axial_DIN0207_L6.3mm_D2.5mm_P7.62mm_Horizontal, F.Cu at (257.8, 119.4)
- added Amp_Fdbk_49: 2M, Resistor_THT:R_Axial_DIN0207_L6.3mm_D2.5mm_P7.62mm_Horizontal, F.Cu at (210.8, 127.0)
- added Amp_Fdbk_5: 2M, Resistor_THT:R_Axial_DIN0207_L6.3mm_D2.5mm_P7.62mm_Horizontal, F.Cu at (246.4, 50.8)
- added Amp_Fdbk_50: 2M, Resistor_THT:R_Axial_DIN0207_L6.3mm_D2.5mm_P7.62mm_Horizontal, F.Cu at (210.8, 132.1)
- added Amp_Fdbk_51: 2M, Resistor_THT:R_Axial_DIN0207_L6.3mm_D2.5mm_P7.62mm_Horizontal, F.Cu at (222.2, 127.0)
- added Amp_Fdbk_52: 2M, Resistor_THT:R_Axial_DIN0207_L6.3mm_D2.5mm_P7.62mm_Horizontal, F.Cu at (222.2, 132.1)
- added Amp_Fdbk_53: 2M, Resistor_THT:R_Axial_DIN0207_L6.3mm_D2.5mm_P7.62mm_Horizontal, F.Cu at (246.4, 127.0)
- added Amp_Fdbk_54: 2M, Resistor_THT:R_Axial_DIN0207_L6.3mm_D2.5mm_P7.62mm_Horizontal, F.Cu at (246.4, 132.1)
- added Amp_Fdbk_55: 2M, Resistor_THT:R_Axial_DIN0207_L6.3mm_D2.5mm_P7.62mm_Horizontal, F.Cu at (257.8, 127.0)
- added Amp_Fdbk_56: 2M, Resistor_THT:R_Axial_DIN0207_L6.3mm_D2.5mm_P7.62mm_Horizontal, F.Cu at (257.8, 132.1)
- added Amp_Fdbk_57: 2M, Resistor_THT:R_Axial_DIN0207_L6.3mm_D2.5mm_P7.62mm_Horizontal, F.Cu at (210.8, 139.7)
- added Amp_Fdbk_58: 2M, Resistor_THT:R_Axial_DIN0207_L6.3mm_D2.5mm_P7.62mm_Horizontal, F.Cu at (210.8, 144.8)
- added Amp_Fdbk_59: 2M, Resistor_THT:R_Axial_DIN0207_L6.3mm_D2.5mm_P7.62mm_Horizontal, F.Cu at (222.2, 139.7)
- added Amp_Fdbk_6: 2M, Resistor_THT:R_Axial_DIN0207_L6.3mm_D2.5mm_P7.62mm_Horizontal, F.Cu at (246.4, 55.9)
- added Amp_Fdbk_60: 2M, Resistor_THT:R_Axial_DIN0207_L6.3mm_D2.5mm_P7.62mm_Horizontal, F.Cu at (222.2, 144.8)
- added Amp_Fdbk_61: 2M, Resistor_THT:R_Axial_DIN0207_L6.3mm_D2.5mm_P7.62mm_Horizontal, F.Cu at (246.4, 139.7)
- added Amp_Fdbk_62: 2M, Resistor_THT:R_Axial_DIN0207_L6.3mm_D2.5mm_P7.62mm_Horizontal, F.Cu at (246.4, 144.8)
- added Amp_Fdbk_63: 2M, Resistor_THT:R_Axial_DIN0207_L6.3mm_D2.5mm_P7.62mm_Horizontal, F.Cu at (257.8, 139.7)
- added Amp_Fdbk_64: 2M, Resistor_THT:R_Axial_DIN0207_L6.3mm_D2.5mm_P7.62mm_Horizontal, F.Cu at (257.8, 144.8)
- added Amp_Fdbk_7: 2M, Resistor_THT:R_Axial_DIN0207_L6.3mm_D2.5mm_P7.62mm_Horizontal, F.Cu at (257.8, 50.8)
- added Amp_Fdbk_8: 2M, Resistor_THT:R_Axial_DIN0207_L6.3mm_D2.5mm_P7.62mm_Horizontal, F.Cu at (257.8, 55.9)
- added Amp_Fdbk_9: 2M, Resistor_THT:R_Axial_DIN0207_L6.3mm_D2.5mm_P7.62mm_Horizontal, F.Cu at (210.9, 63.5)
- added DEMUX_1: 74HC138D-Q100,118, DEMUX:footprints, F.Cu at (317.5, 83.8)
- added Drv_I_Sel_1: 2K, Resistor_THT:R_Axial_DIN0207_L6.3mm_D2.5mm_P7.62mm_Horizontal, F.Cu at (284.5, 50.8)
- added Drv_I_Sel_2: 2K, Resistor_THT:R_Axial_DIN0207_L6.3mm_D2.5mm_P7.62mm_Horizontal, F.Cu at (284.5, 63.5)
- added Drv_I_Sel_3: 2K, Resistor_THT:R_Axial_DIN0207_L6.3mm_D2.5mm_P7.62mm_Horizontal, F.Cu at (284.5, 76.2)
- added Drv_I_Sel_4: 2K, Resistor_THT:R_Axial_DIN0207_L6.3mm_D2.5mm_P7.62mm_Horizontal, F.Cu at (284.5, 88.9)
- added Drv_I_Sel_5: 2K, Resistor_THT:R_Axial_DIN0207_L6.3mm_D2.5mm_P7.62mm_Horizontal, F.Cu at (284.5, 101.6)
- added Drv_I_Sel_6: 2K, Resistor_THT:R_Axial_DIN0207_L6.3mm_D2.5mm_P7.62mm_Horizontal, F.Cu at (284.5, 114.3)
- added Drv_I_Sel_7: 2K, Resistor_THT:R_Axial_DIN0207_L6.3mm_D2.5mm_P7.62mm_Horizontal, F.Cu at (284.5, 127.0)
- added Drv_I_Sel_8: 2K, Resistor_THT:R_Axial_DIN0207_L6.3mm_D2.5mm_P7.62mm_Horizontal, F.Cu at (284.5, 139.7)
- added Drv_RST_PU_1: 10K, Resistor_THT:R_Axial_DIN0207_L6.3mm_D2.5mm_P7.62mm_Horizontal, F.Cu at (284.5, 55.9)
- added Drv_RST_PU_2: 10K, Resistor_THT:R_Axial_DIN0207_L6.3mm_D2.5mm_P7.62mm_Horizontal, F.Cu at (284.5, 68.6)
- added Drv_RST_PU_3: 10K, Resistor_THT:R_Axial_DIN0207_L6.3mm_D2.5mm_P7.62mm_Horizontal, F.Cu at (284.5, 81.3)
- added Drv_RST_PU_4: 10K, Resistor_THT:R_Axial_DIN0207_L6.3mm_D2.5mm_P7.62mm_Horizontal, F.Cu at (284.5, 94.0)
- added Drv_RST_PU_5: 10K, Resistor_THT:R_Axial_DIN0207_L6.3mm_D2.5mm_P7.62mm_Horizontal, F.Cu at (284.5, 106.7)
- added Drv_RST_PU_6: 10K, Resistor_THT:R_Axial_DIN0207_L6.3mm_D2.5mm_P7.62mm_Horizontal, F.Cu at (284.5, 119.4)
- added Drv_RST_PU_7: 10K, Resistor_THT:R_Axial_DIN0207_L6.3mm_D2.5mm_P7.62mm_Horizontal, F.Cu at (284.5, 132.1)
- added Drv_RST_PU_8: 10K, Resistor_THT:R_Axial_DIN0207_L6.3mm_D2.5mm_P7.62mm_Horizontal, F.Cu at (284.5, 144.8)
- added LD1: WP154A4SEJ3VBDZGC/CA, RGB LED:WP154A4SEJ3VBDZGC&slash_CA, F.Cu at (27.9, 71.1)
- added LD10: WP154A4SEJ3VBDZGC/CA, RGB LED:WP154A4SEJ3VBDZGC&slash_CA, F.Cu at (35.6, 78.7)
- added LD11: WP154A4SEJ3VBDZGC/CA, RGB LED:WP154A4SEJ3VBDZGC&slash_CA, F.Cu at (43.2, 78.7)
- added LD12: WP154A4SEJ3VBDZGC/CA, RGB LED:WP154A4SEJ3VBDZGC&slash_CA, F.Cu at (50.8, 78.7)
- added LD13: WP154A4SEJ3VBDZGC/CA, RGB LED:WP154A4SEJ3VBDZGC&slash_CA, F.Cu at (58.4, 78.7)
- added LD14: WP154A4SEJ3VBDZGC/CA, RGB LED:WP154A4SEJ3VBDZGC&slash_CA, F.Cu at (66.0, 78.7)
- added LD15: WP154A4SEJ3VBDZGC/CA, RGB LED:WP154A4SEJ3VBDZGC&slash_CA, F.Cu at (73.7, 78.7)
- added LD16: WP154A4SEJ3VBDZGC/CA, RGB LED:WP154A4SEJ3VBDZGC&slash_CA, F.Cu at (81.3, 78.7)
- added LD17: WP154A4SEJ3VBDZGC/CA, RGB LED:WP154A4SEJ3VBDZGC&slash_CA, F.Cu at (27.9, 86.4)
- added LD18: WP154A4SEJ3VBDZGC/CA, RGB LED:WP154A4SEJ3VBDZGC&slash_CA, F.Cu at (35.6, 86.4)
- added LD19: WP154A4SEJ3VBDZGC/CA, RGB LED:WP154A4SEJ3VBDZGC&slash_CA, F.Cu at (43.2, 86.4)
- added LD2: WP154A4SEJ3VBDZGC/CA, RGB LED:WP154A4SEJ3VBDZGC&slash_CA, F.Cu at (35.6, 71.1)
- added LD20: WP154A4SEJ3VBDZGC/CA, RGB LED:WP154A4SEJ3VBDZGC&slash_CA, F.Cu at (50.8, 86.4)
- added LD21: WP154A4SEJ3VBDZGC/CA, RGB LED:WP154A4SEJ3VBDZGC&slash_CA, F.Cu at (58.4, 86.4)
- added LD22: WP154A4SEJ3VBDZGC/CA, RGB LED:WP154A4SEJ3VBDZGC&slash_CA, F.Cu at (66.0, 86.4)
- added LD23: WP154A4SEJ3VBDZGC/CA, RGB LED:WP154A4SEJ3VBDZGC&slash_CA, F.Cu at (73.7, 86.4)
- added LD24: WP154A4SEJ3VBDZGC/CA, RGB LED:WP154A4SEJ3VBDZGC&slash_CA, F.Cu at (81.3, 86.4)
- added LD25: WP154A4SEJ3VBDZGC/CA, RGB LED:WP154A4SEJ3VBDZGC&slash_CA, F.Cu at (27.9, 94.0)
- added LD26: WP154A4SEJ3VBDZGC/CA, RGB LED:WP154A4SEJ3VBDZGC&slash_CA, F.Cu at (35.6, 94.0)
- added LD27: WP154A4SEJ3VBDZGC/CA, RGB LED:WP154A4SEJ3VBDZGC&slash_CA, F.Cu at (43.2, 94.0)
- added LD28: WP154A4SEJ3VBDZGC/CA, RGB LED:WP154A4SEJ3VBDZGC&slash_CA, F.Cu at (50.8, 94.0)
- added LD29: WP154A4SEJ3VBDZGC/CA, RGB LED:WP154A4SEJ3VBDZGC&slash_CA, F.Cu at (58.4, 94.0)
- added LD3: WP154A4SEJ3VBDZGC/CA, RGB LED:WP154A4SEJ3VBDZGC&slash_CA, F.Cu at (43.2, 71.1)
- added LD30: WP154A4SEJ3VBDZGC/CA, RGB LED:WP154A4SEJ3VBDZGC&slash_CA, F.Cu at (66.0, 94.0)
- added LD31: WP154A4SEJ3VBDZGC/CA, RGB LED:WP154A4SEJ3VBDZGC&slash_CA, F.Cu at (73.7, 94.0)
- added LD32: WP154A4SEJ3VBDZGC/CA, RGB LED:WP154A4SEJ3VBDZGC&slash_CA, F.Cu at (81.3, 94.0)
- added LD33: WP154A4SEJ3VBDZGC/CA, RGB LED:WP154A4SEJ3VBDZGC&slash_CA, F.Cu at (27.9, 101.6)
- added LD34: WP154A4SEJ3VBDZGC/CA, RGB LED:WP154A4SEJ3VBDZGC&slash_CA, F.Cu at (35.6, 101.6)
- added LD35: WP154A4SEJ3VBDZGC/CA, RGB LED:WP154A4SEJ3VBDZGC&slash_CA, F.Cu at (43.2, 101.6)
- added LD36: WP154A4SEJ3VBDZGC/CA, RGB LED:WP154A4SEJ3VBDZGC&slash_CA, F.Cu at (50.8, 101.6)
- added LD37: WP154A4SEJ3VBDZGC/CA, RGB LED:WP154A4SEJ3VBDZGC&slash_CA, F.Cu at (58.4, 101.6)
- added LD38: WP154A4SEJ3VBDZGC/CA, RGB LED:WP154A4SEJ3VBDZGC&slash_CA, F.Cu at (66.0, 101.6)
- added LD39: WP154A4SEJ3VBDZGC/CA, RGB LED:WP154A4SEJ3VBDZGC&slash_CA, F.Cu at (73.7, 101.6)
- added LD4: WP154A4SEJ3VBDZGC/CA, RGB LED:WP154A4SEJ3VBDZGC&slash_CA, F.Cu at (50.8, 71.1)
- added LD40: WP154A4SEJ3VBDZGC/CA, RGB LED:WP154A4SEJ3VBDZGC&slash_CA, F.Cu at (81.3, 101.6)
- added LD41: WP154A4SEJ3VBDZGC/CA, RGB LED:WP154A4SEJ3VBDZGC&slash_CA, F.Cu at (27.9, 109.2)
- added LD42: WP154A4SEJ3VBDZGC/CA, RGB LED:WP154A4SEJ3VBDZGC&slash_CA, F.Cu at (35.6, 109.2)
- added LD43: WP154A4SEJ3VBDZGC/CA, RGB LED:WP154A4SEJ3VBDZGC&slash_CA, F.Cu at (43.2, 109.2)
- added LD44: WP154A4SEJ3VBDZGC/CA, RGB LED:WP154A4SEJ3VBDZGC&slash_CA, F.Cu at (50.8, 109.2)
- added LD45: WP154A4SEJ3VBDZGC/CA, RGB LED:WP154A4SEJ3VBDZGC&slash_CA, F.Cu at (58.4, 109.2)
- added LD46: WP154A4SEJ3VBDZGC/CA, RGB LED:WP154A4SEJ3VBDZGC&slash_CA, F.Cu at (66.0, 109.2)
- added LD47: WP154A4SEJ3VBDZGC/CA, RGB LED:WP154A4SEJ3VBDZGC&slash_CA, F.Cu at (73.7, 109.2)
- added LD48: WP154A4SEJ3VBDZGC/CA, RGB LED:WP154A4SEJ3VBDZGC&slash_CA, F.Cu at (81.3, 109.2)
- added LD49: WP154A4SEJ3VBDZGC/CA, RGB LED:WP154A4SEJ3VBDZGC&slash_CA, F.Cu at (27.9, 116.8)
- added LD5: WP154A4SEJ3VBDZGC/CA, RGB LED:WP154A4SEJ3VBDZGC&slash_CA, F.Cu at (58.4, 71.1)
- added LD50: WP154A4SEJ3VBDZGC/CA, RGB LED:WP154A4SEJ3VBDZGC&slash_CA, F.Cu at (35.6, 116.8)
- added LD51: WP154A4SEJ3VBDZGC/CA, RGB LED:WP154A4SEJ3VBDZGC&slash_CA, F.Cu at (43.2, 116.8)
- added LD52: WP154A4SEJ3VBDZGC/CA, RGB LED:WP154A4SEJ3VBDZGC&slash_CA, F.Cu at (50.8, 116.8)
- added LD53: WP154A4SEJ3VBDZGC/CA, RGB LED:WP154A4SEJ3VBDZGC&slash_CA, F.Cu at (58.4, 116.8)
- added LD54: WP154A4SEJ3VBDZGC/CA, RGB LED:WP154A4SEJ3VBDZGC&slash_CA, F.Cu at (66.0, 116.8)
- added LD55: WP154A4SEJ3VBDZGC/CA, RGB LED:WP154A4SEJ3VBDZGC&slash_CA, F.Cu at (73.7, 116.8)
- added LD56: WP154A4SEJ3VBDZGC/CA, RGB LED:WP154A4SEJ3VBDZGC&slash_CA, F.Cu at (81.3, 116.8)
- added LD57: WP154A4SEJ3VBDZGC/CA, RGB LED:WP154A4SEJ3VBDZGC&slash_CA, F.Cu at (27.9, 124.5)
- added LD58: WP154A4SEJ3VBDZGC/CA, RGB LED:WP154A4SEJ3VBDZGC&slash_CA, F.Cu at (35.6, 124.5)
- added LD59: WP154A4SEJ3VBDZGC/CA, RGB LED:WP154A4SEJ3VBDZGC&slash_CA, F.Cu at (43.2, 124.5)
- added LD6: WP154A4SEJ3VBDZGC/CA, RGB LED:WP154A4SEJ3VBDZGC&slash_CA, F.Cu at (66.0, 71.1)
- added LD60: WP154A4SEJ3VBDZGC/CA, RGB LED:WP154A4SEJ3VBDZGC&slash_CA, F.Cu at (50.8, 124.5)
- added LD61: WP154A4SEJ3VBDZGC/CA, RGB LED:WP154A4SEJ3VBDZGC&slash_CA, F.Cu at (58.4, 124.5)
- added LD62: WP154A4SEJ3VBDZGC/CA, RGB LED:WP154A4SEJ3VBDZGC&slash_CA, F.Cu at (66.0, 124.5)
- added LD63: WP154A4SEJ3VBDZGC/CA, RGB LED:WP154A4SEJ3VBDZGC&slash_CA, F.Cu at (73.7, 124.5)
- added LD64: WP154A4SEJ3VBDZGC/CA, RGB LED:WP154A4SEJ3VBDZGC&slash_CA, F.Cu at (81.3, 124.5)
- added LD7: WP154A4SEJ3VBDZGC/CA, RGB LED:WP154A4SEJ3VBDZGC&slash_CA, F.Cu at (73.7, 71.1)
- added LD8: WP154A4SEJ3VBDZGC/CA, RGB LED:WP154A4SEJ3VBDZGC&slash_CA, F.Cu at (81.3, 71.1)
- added LD9: WP154A4SEJ3VBDZGC/CA, RGB LED:WP154A4SEJ3VBDZGC&slash_CA, F.Cu at (27.9, 78.7)
- added LED_Driver_1: PCA9956BTWY, LED Driver:SOP50P640X110-39N, F.Cu at (276.9, 53.3)
- added LED_Driver_2: PCA9956BTWY, LED Driver:SOP50P640X110-39N, F.Cu at (276.9, 66.0)
- added LED_Driver_3: PCA9956BTWY, LED Driver:SOP50P640X110-39N, F.Cu at (276.9, 78.7)
- added LED_Driver_4: PCA9956BTWY, LED Driver:SOP50P640X110-39N, F.Cu at (276.9, 91.4)
- added LED_Driver_5: PCA9956BTWY, LED Driver:SOP50P640X110-39N, F.Cu at (276.8, 104.1)
- added LED_Driver_6: PCA9956BTWY, LED Driver:SOP50P640X110-39N, F.Cu at (276.8, 116.8)
- added LED_Driver_7: PCA9956BTWY, LED Driver:SOP50P640X110-39N, F.Cu at (276.9, 129.5)
- added LED_Driver_8: PCA9956BTWY, LED Driver:SOP50P640X110-39N, F.Cu at (276.9, 142.2)
- added Lvl_Sftr_1: VSSOP8_SOT765-1_NEX, Level Shifter:LSF0102DCH, F.Cu at (317.5, 111.8)
- added OC1: CPC1125N, Opto-coupler:footprints, F.Cu at (94.0, 53.3)
- added OC10: CPC1125N, Opto-coupler:footprints, F.Cu at (104.1, 66.0)
- added OC11: CPC1125N, Opto-coupler:footprints, F.Cu at (114.3, 66.0)
- added OC12: CPC1125N, Opto-coupler:footprints, F.Cu at (124.5, 66.0)
- added OC13: CPC1125N, Opto-coupler:footprints, F.Cu at (134.6, 66.0)
- added OC14: CPC1125N, Opto-coupler:footprints, F.Cu at (144.8, 66.0)
- added OC15: CPC1125N, Opto-coupler:footprints, F.Cu at (154.9, 66.0)
- added OC16: CPC1125N, Opto-coupler:footprints, F.Cu at (165.1, 66.0)
- added OC17: CPC1125N, Opto-coupler:footprints, F.Cu at (94.0, 78.7)
- added OC18: CPC1125N, Opto-coupler:footprints, F.Cu at (104.1, 78.7)
- added OC19: CPC1125N, Opto-coupler:footprints, F.Cu at (114.3, 78.7)
- added OC2: CPC1125N, Opto-coupler:footprints, F.Cu at (104.1, 53.3)
- added OC20: CPC1125N, Opto-coupler:footprints, F.Cu at (124.5, 78.7)
- added OC21: CPC1125N, Opto-coupler:footprints, F.Cu at (134.6, 78.7)
- added OC22: CPC1125N, Opto-coupler:footprints, F.Cu at (144.8, 78.7)
- added OC23: CPC1125N, Opto-coupler:footprints, F.Cu at (154.9, 78.7)
- added OC24: CPC1125N, Opto-coupler:footprints, F.Cu at (165.1, 78.7)
- added OC25: CPC1125N, Opto-coupler:footprints, F.Cu at (94.0, 91.4)
- added OC26: CPC1125N, Opto-coupler:footprints, F.Cu at (104.1, 91.4)
- added OC27: CPC1125N, Opto-coupler:footprints, F.Cu at (114.3, 91.4)
- added OC28: CPC1125N, Opto-coupler:footprints, F.Cu at (124.5, 91.4)
- added OC29: CPC1125N, Opto-coupler:footprints, F.Cu at (134.6, 91.4)
- added OC3: CPC1125N, Opto-coupler:footprints, F.Cu at (114.3, 53.3)
- added OC30: CPC1125N, Opto-coupler:footprints, F.Cu at (144.8, 91.4)
- added OC31: CPC1125N, Opto-coupler:footprints, F.Cu at (154.9, 91.4)
- added OC32: CPC1125N, Opto-coupler:footprints, F.Cu at (165.1, 91.4)
- added OC33: CPC1125N, Opto-coupler:footprints, F.Cu at (94.0, 104.1)
- added OC34: CPC1125N, Opto-coupler:footprints, F.Cu at (104.1, 104.1)
- added OC35: CPC1125N, Opto-coupler:footprints, F.Cu at (114.3, 104.1)
- added OC36: CPC1125N, Opto-coupler:footprints, F.Cu at (124.5, 104.1)
- added OC37: CPC1125N, Opto-coupler:footprints, F.Cu at (134.6, 104.1)
- added OC38: CPC1125N, Opto-coupler:footprints, F.Cu at (144.8, 104.1)
- added OC39: CPC1125N, Opto-coupler:footprints, F.Cu at (154.9, 104.1)
- added OC4: CPC1125N, Opto-coupler:footprints, F.Cu at (124.5, 53.3)
- added OC40: CPC1125N, Opto-coupler:footprints, F.Cu at (165.1, 104.1)
- added OC41: CPC1125N, Opto-coupler:footprints, F.Cu at (94.0, 116.8)
- added OC42: CPC1125N, Opto-coupler:footprints, F.Cu at (104.1, 116.8)
- added OC43: CPC1125N, Opto-coupler:footprints, F.Cu at (114.3, 116.8)
- added OC44: CPC1125N, Opto-coupler:footprints, F.Cu at (124.5, 116.8)
- added OC45: CPC1125N, Opto-coupler:footprints, F.Cu at (134.6, 116.8)
- added OC46: CPC1125N, Opto-coupler:footprints, F.Cu at (144.8, 116.8)
- added OC47: CPC1125N, Opto-coupler:footprints, F.Cu at (154.9, 116.8)
- added OC48: CPC1125N, Opto-coupler:footprints, F.Cu at (165.1, 116.8)
- added OC49: CPC1125N, Opto-coupler:footprints, F.Cu at (94.0, 129.5)
- added OC5: CPC1125N, Opto-coupler:footprints, F.Cu at (134.6, 53.3)
- added OC50: CPC1125N, Opto-coupler:footprints, F.Cu at (104.1, 129.5)
- added OC51: CPC1125N, Opto-coupler:footprints, F.Cu at (114.3, 129.5)
- added OC52: CPC1125N, Opto-coupler:footprints, F.Cu at (124.5, 129.5)
- added OC53: CPC1125N, Opto-coupler:footprints, F.Cu at (134.6, 129.5)
- added OC54: CPC1125N, Opto-coupler:footprints, F.Cu at (144.8, 129.5)
- added OC55: CPC1125N, Opto-coupler:footprints, F.Cu at (154.9, 129.5)
- added OC56: CPC1125N, Opto-coupler:footprints, F.Cu at (165.1, 129.5)
- added OC57: CPC1125N, Opto-coupler:footprints, F.Cu at (94.0, 142.2)
- added OC58: CPC1125N, Opto-coupler:footprints, F.Cu at (104.1, 142.2)
- added OC59: CPC1125N, Opto-coupler:footprints, F.Cu at (114.3, 142.2)
- added OC6: CPC1125N, Opto-coupler:footprints, F.Cu at (144.8, 53.3)
- added OC60: CPC1125N, Opto-coupler:footprints, F.Cu at (124.5, 142.2)
- added OC61: CPC1125N, Opto-coupler:footprints, F.Cu at (134.6, 142.2)
- added OC62: CPC1125N, Opto-coupler:footprints, F.Cu at (144.8, 142.2)
- added OC63: CPC1125N, Opto-coupler:footprints, F.Cu at (154.9, 142.2)
- added OC64: CPC1125N, Opto-coupler:footprints, F.Cu at (165.1, 142.2)
- added OC7: CPC1125N, Opto-coupler:footprints, F.Cu at (154.9, 53.3)
- added OC8: CPC1125N, Opto-coupler:footprints, F.Cu at (165.1, 53.3)
- added OC9: CPC1125N, Opto-coupler:footprints, F.Cu at (94.0, 66.0)
- added Pin_Header_1: Conn_02x16_Odd_Even, Connector_PinHeader_2.54mm:PinHeader_2x16_P2.54mm_Vertical, F.Cu at (334.0, 77.5)
- added Rev_Bias_Sel_1: 100K, Potentiometer_THT:Potentiometer_Runtron_RM-065_Vertical, F.Cu at (315.0, 96.5)
Other:
- board outline added: 324.7 x 110.9 mm

Commit message: Rearranged PCB Components
Parts:
- Lvl_Sftr_1: value VSSOP8_SOT765-1_NEX -> LSF0102DCH
- moved Amp_Fdbk_8 119.4 mm to (174.0, -29.2), turned to 90 degrees
- moved Amp_Fdbk_61 117.6 mm to (174.0, 232.4), turned to 90 degrees
- moved Amp_Fdbk_4 112.5 mm to (148.6, -29.2), turned to 90 degrees
- moved Amp_Fdbk_57 111.7 mm to (148.6, 232.4), turned to 90 degrees
- moved Amp_Fdbk_64 110.8 mm to (174.0, 217.2), turned to 90 degrees
- moved OC57 106.7 mm to (154.9, 229.9), turned to 90 degrees
- moved OC58 103.9 mm to (160.0, 229.9), turned to 90 degrees
- moved Amp_Fdbk_7 103.7 mm to (191.8, -29.2), turned to 90 degrees
- moved Amp_Fdbk_60 103.3 mm to (148.6, 217.2), turned to 90 degrees
- moved Amp_Fdbk_62 103.3 mm to (191.8, 232.4), turned to 90 degrees
- moved Amp_Fdbk_63 101.8 mm to (191.8, 217.2), turned to 90 degrees
- moved Amp_Fdbk_16 101.4 mm to (174.0, 11.5), turned to 90 degrees
- moved OC3 98.8 mm to (160.0, -34.3), turned to -90 degrees
- moved OC61 98.8 mm to (180.3, 229.9), turned to 90 degrees
- moved Amp_Fdbk_58 98.3 mm to (166.4, 232.4), turned to 90 degrees
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Connections:
- Amp_Fdbk_1 pad 1: /LED Row IO 1/ LDRow_Amps/Amp_OP_1 -> /LED Row IO 1/ LDRow_Amps/Amp_IP_1
- Amp_Fdbk_1 pad 2: /LED Row IO 1/ LDRow_Amps/Amp_IP_1 -> /LED Row IO 1/ LDRow_Amps/Amp_OP_1
- Amp_Fdbk_10 pad 1: /LED Row IO 2/ LDRow_Amps/Amp_OP_2 -> /LED Row IO 2/ LDRow_Amps/Amp_IP_2
- Amp_Fdbk_10 pad 2: /LED Row IO 2/ LDRow_Amps/Amp_IP_2 -> /LED Row IO 2/ LDRow_Amps/Amp_OP_2
- Amp_Fdbk_13 pad 1: /LED Row IO 2/ LDRow_Amps/Amp_OP_5 -> /LED Row IO 2/ LDRow_Amps/Amp_IP_5
- Amp_Fdbk_13 pad 2: /LED Row IO 2/ LDRow_Amps/Amp_IP_5 -> /LED Row IO 2/ LDRow_Amps/Amp_OP_5
- Amp_Fdbk_14 pad 1: /LED Row IO 2/ LDRow_Amps/Amp_OP_6 -> /LED Row IO 2/ LDRow_Amps/Amp_IP_6
- Amp_Fdbk_14 pad 2: /LED Row IO 2/ LDRow_Amps/Amp_IP_6 -> /LED Row IO 2/ LDRow_Amps/Amp_OP_6
- Amp_Fdbk_17 pad 1: /LED Row IO 3/ LDRow_Amps/Amp_OP_1 -> /LED Row IO 3/ LDRow_Amps/Amp_IP_1
- Amp_Fdbk_17 pad 2: /LED Row IO 3/ LDRow_Amps/Amp_IP_1 -> /LED Row IO 3/ LDRow_Amps/Amp_OP_1
- Amp_Fdbk_18 pad 1: /LED Row IO 3/ LDRow_Amps/Amp_OP_2 -> /LED Row IO 3/ LDRow_Amps/Amp_IP_2
- Amp_Fdbk_18 pad 2: /LED Row IO 3/ LDRow_Amps/Amp_IP_2 -> /LED Row IO 3/ LDRow_Amps/Amp_OP_2
- Amp_Fdbk_2 pad 1: /LED Row IO 1/ LDRow_Amps/Amp_OP_2 -> /LED Row IO 1/ LDRow_Amps/Amp_IP_2
- Amp_Fdbk_2 pad 2: /LED Row IO 1/ LDRow_Amps/Amp_IP_2 -> /LED Row IO 1/ LDRow_Amps/Amp_OP_2
- Amp_Fdbk_21 pad 1: /LED Row IO 3/ LDRow_Amps/Amp_OP_5 -> /LED Row IO 3/ LDRow_Amps/Amp_IP_5
- Amp_Fdbk_21 pad 2: /LED Row IO 3/ LDRow_Amps/Amp_IP_5 -> /LED Row IO 3/ LDRow_Amps/Amp_OP_5
- Amp_Fdbk_22 pad 1: /LED Row IO 3/ LDRow_Amps/Amp_OP_6 -> /LED Row IO 3/ LDRow_Amps/Amp_IP_6
- Amp_Fdbk_22 pad 2: /LED Row IO 3/ LDRow_Amps/Amp_IP_6 -> /LED Row IO 3/ LDRow_Amps/Amp_OP_6
- Amp_Fdbk_25 pad 1: /LED Row IO 4/ LDRow_Amps/Amp_OP_1 -> /LED Row IO 4/ LDRow_Amps/Amp_IP_1
- Amp_Fdbk_25 pad 2: /LED Row IO 4/ LDRow_Amps/Amp_IP_1 -> /LED Row IO 4/ LDRow_Amps/Amp_OP_1
- Amp_Fdbk_26 pad 1: /LED Row IO 4/ LDRow_Amps/Amp_OP_2 -> /LED Row IO 4/ LDRow_Amps/Amp_IP_2
- Amp_Fdbk_26 pad 2: /LED Row IO 4/ LDRow_Amps/Amp_IP_2 -> /LED Row IO 4/ LDRow_Amps/Amp_OP_2
- Amp_Fdbk_29 pad 1: /LED Row IO 4/ LDRow_Amps/Amp_OP_5 -> /LED Row IO 4/ LDRow_Amps/Amp_IP_5
- Amp_Fdbk_29 pad 2: /LED Row IO 4/ LDRow_Amps/Amp_IP_5 -> /LED Row IO 4/ LDRow_Amps/Amp_OP_5
- Amp_Fdbk_30 pad 1: /LED Row IO 4/ LDRow_Amps/Amp_OP_6 -> /LED Row IO 4/ LDRow_Amps/Amp_IP_6
- Amp_Fdbk_30 pad 2: /LED Row IO 4/ LDRow_Amps/Amp_IP_6 -> /LED Row IO 4/ LDRow_Amps/Amp_OP_6
- Amp_Fdbk_33 pad 1: /LED Row IO 5/ LDRow_Amps/Amp_OP_1 -> /LED Row IO 5/ LDRow_Amps/Amp_IP_1
- Amp_Fdbk_33 pad 2: /LED Row IO 5/ LDRow_Amps/Amp_IP_1 -> /LED Row IO 5/ LDRow_Amps/Amp_OP_1
- Amp_Fdbk_34 pad 1: /LED Row IO 5/ LDRow_Amps/Amp_OP_2 -> /LED Row IO 5/ LDRow_Amps/Amp_IP_2
- Amp_Fdbk_34 pad 2: /LED Row IO 5/ LDRow_Amps/Amp_IP_2 -> /LED Row IO 5/ LDRow_Amps/Amp_OP_2
- Amp_Fdbk_37 pad 1: /LED Row IO 5/ LDRow_Amps/Amp_OP_5 -> /LED Row IO 5/ LDRow_Amps/Amp_IP_5
- Amp_Fdbk_37 pad 2: /LED Row IO 5/ LDRow_Amps/Amp_IP_5 -> /LED Row IO 5/ LDRow_Amps/Amp_OP_5
- Amp_Fdbk_38 pad 1: /LED Row IO 5/ LDRow_Amps/Amp_OP_6 -> /LED Row IO 5/ LDRow_Amps/Amp_IP_6
- Amp_Fdbk_38 pad 2: /LED Row IO 5/ LDRow_Amps/Amp_IP_6 -> /LED Row IO 5/ LDRow_Amps/Amp_OP_6
- Amp_Fdbk_41 pad 1: /LED Row IO 6/ LDRow_Amps/Amp_OP_1 -> /LED Row IO 6/ LDRow_Amps/Amp_IP_1
- Amp_Fdbk_41 pad 2: /LED Row IO 6/ LDRow_Amps/Amp_IP_1 -> /LED Row IO 6/ LDRow_Amps/Amp_OP_1
- Amp_Fdbk_42 pad 1: /LED Row IO 6/ LDRow_Amps/Amp_OP_2 -> /LED Row IO 6/ LDRow_Amps/Amp_IP_2
- Amp_Fdbk_42 pad 2: /LED Row IO 6/ LDRow_Amps/Amp_IP_2 -> /LED Row IO 6/ LDRow_Amps/Amp_OP_2
- Amp_Fdbk_45 pad 1: /LED Row IO 6/ LDRow_Amps/Amp_OP_5 -> /LED Row IO 6/ LDRow_Amps/Amp_IP_5
- Amp_Fdbk_45 pad 2: /LED Row IO 6/ LDRow_Amps/Amp_IP_5 -> /LED Row IO 6/ LDRow_Amps/Amp_OP_5
- Amp_Fdbk_46 pad 1: /LED Row IO 6/ LDRow_Amps/Amp_OP_6 -> /LED Row IO 6/ LDRow_Amps/Amp_IP_6
- Amp_Fdbk_46 pad 2: /LED Row IO 6/ LDRow_Amps/Amp_IP_6 -> /LED Row IO 6/ LDRow_Amps/Amp_OP_6
- Amp_Fdbk_49 pad 1: /LED Row IO 7/ LDRow_Amps/Amp_OP_1 -> /LED Row IO 7/ LDRow_Amps/Amp_IP_1
- Amp_Fdbk_49 pad 2: /LED Row IO 7/ LDRow_Amps/Amp_IP_1 -> /LED Row IO 7/ LDRow_Amps/Amp_OP_1
- Amp_Fdbk_5 pad 1: /LED Row IO 1/ LDRow_Amps/Amp_OP_5 -> /LED Row IO 1/ LDRow_Amps/Amp_IP_5
- Amp_Fdbk_5 pad 2: /LED Row IO 1/ LDRow_Amps/Amp_IP_5 -> /LED Row IO 1/ LDRow_Amps/Amp_OP_5
- Amp_Fdbk_50 pad 1: /LED Row IO 7/ LDRow_Amps/Amp_OP_2 -> /LED Row IO 7/ LDRow_Amps/Amp_IP_2
- Amp_Fdbk_50 pad 2: /LED Row IO 7/ LDRow_Amps/Amp_IP_2 -> /LED Row IO 7/ LDRow_Amps/Amp_OP_2
- Amp_Fdbk_53 pad 1: /LED Row IO 7/ LDRow_Amps/Amp_OP_5 -> /LED Row IO 7/ LDRow_Amps/Amp_IP_5
- Amp_Fdbk_53 pad 2: /LED Row IO 7/ LDRow_Amps/Amp_IP_5 -> /LED Row IO 7/ LDRow_Amps/Amp_OP_5
- Amp_Fdbk_54 pad 1: /LED Row IO 7/ LDRow_Amps/Amp_OP_6 -> /LED Row IO 7/ LDRow_Amps/Amp_IP_6
- Amp_Fdbk_54 pad 2: /LED Row IO 7/ LDRow_Amps/Amp_IP_6 -> /LED Row IO 7/ LDRow_Amps/Amp_OP_6
- Amp_Fdbk_57 pad 1: /LED Row IO 8/ LDRow_Amps/Amp_OP_1 -> /LED Row IO 8/ LDRow_Amps/Amp_IP_1
- Amp_Fdbk_57 pad 2: /LED Row IO 8/ LDRow_Amps/Amp_IP_1 -> /LED Row IO 8/ LDRow_Amps/Amp_OP_1
- Amp_Fdbk_58 pad 1: /LED Row IO 8/ LDRow_Amps/Amp_OP_2 -> /LED Row IO 8/ LDRow_Amps/Amp_IP_2
- Amp_Fdbk_58 pad 2: /LED Row IO 8/ LDRow_Amps/Amp_IP_2 -> /LED Row IO 8/ LDRow_Amps/Amp_OP_2
- Amp_Fdbk_6 pad 1: /LED Row IO 1/ LDRow_Amps/Amp_OP_6 -> /LED Row IO 1/ LDRow_Amps/Amp_IP_6
- Amp_Fdbk_6 pad 2: /LED Row IO 1/ LDRow_Amps/Amp_IP_6 -> /LED Row IO 1/ LDRow_Amps/Amp_OP_6
- Amp_Fdbk_61 pad 1: /LED Row IO 8/ LDRow_Amps/Amp_OP_5 -> /LED Row IO 8/ LDRow_Amps/Amp_IP_5
- Amp_Fdbk_61 pad 2: /LED Row IO 8/ LDRow_Amps/Amp_IP_5 -> /LED Row IO 8/ LDRow_Amps/Amp_OP_5
- Amp_Fdbk_62 pad 1: /LED Row IO 8/ LDRow_Amps/Amp_OP_6 -> /LED Row IO 8/ LDRow_Amps/Amp_IP_6
- Amp_Fdbk_62 pad 2: /LED Row IO 8/ LDRow_Amps/Amp_IP_6 -> /LED Row IO 8/ LDRow_Amps/Amp_OP_6
- Amp_Fdbk_9 pad 1: /LED Row IO 2/ LDRow_Amps/Amp_OP_1 -> /LED Row IO 2/ LDRow_Amps/Amp_IP_1
- Amp_Fdbk_9 pad 2: /LED Row IO 2/ LDRow_Amps/Amp_IP_1 -> /LED Row IO 2/ LDRow_Amps/Amp_OP_1
Other:
- board size 324.7 x 110.9 mm -> 417.4 x 315.4 mm

Commit message: Boundary Change
Other:
- board size 417.4 x 315.4 mm -> 408.6 x 315.4 mm
Changed lines of the file:
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@@
     )
   )
-  (gr_rect (start 17.699693 -59.61) (end 435.149693 255.8) (layer "Edge.Cuts") (width 0.1) (fill none))
+  (gr_rect (start 1.189693 -59.61) (end 409.749693 255.8) (layer "Edge.Cuts") (width 0.1) (fill none))
 )

Commit message: Fixed ADC Orientation
Parts:
- turned ADC_1 to 90 degrees
Changed lines of the file:
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@@
   )
   (footprint "ADC:MCP3008-I&slash_P" (layer "F.Cu")
-    (at 157.48 -5.08 -90)
+    (at 157.48 -5.08 90)
     (property "MPN" "MCP3008-I/P")
     (property "Sheetfile" "led_row_io.kicad_sch")
@@
     (fp_line (start -4.2164 8.4836) (end -4.2164 9.2964) (layer "F.Fab") (width 0.1))
     (fp_arc (start 3.720968 -12.651613) (mid 1.856613 -7.074032) (end -3.720968 -8.938387) (layer "F.Fab") (width 0.1))
-    (pad "1" thru_hole rect (at -3.81 -8.89 270) (size 1.524 1.524) (drill 0.8128) (layers *.Cu *.Mask)
+    (pad "1" thru_hole rect (at -3.81 -8.89 90) (size 1.524 1.524) (drill 0.8128) (layers *.Cu *.Mask)
       (net 8 "/LED Row IO 1/ LDRow_Amps/Amp_OP_1") (pinfunction "CH0") (pintype "input"))
-    (pad "2" thru_hole circle (at -3.81 -6.35 270) (size 1.524 1.524) (drill 0.8128) (layers *.Cu *.Mask)
+    (pad "2" thru_hole circle (at -3.81 -6.35 90) (size 1.524 1.524) (drill 0.8128) (layers *.Cu *.Mask)
       (net 7 "/LED Row IO 1/ LDRow_Amps/Amp_OP_2") (pinfunction "CH1") (pintype "input"))
-    (pad "3" thru_hole circle (at -3.81 -3.81 270) (size 1.524 1.524) (drill 0.8128) (layers *.Cu *.Mask)
+    (pad "3" thru_hole circle (at -3.81 -3.81 90) (size 1.524 1.524) (drill 0.8128) (layers *.Cu *.Mask)
       (net 6 "/LED Row IO 1/ LDRow_Amps/Amp_OP_3") (pinfunction "CH2") (pintype "input"))
-    (pad "4" thru_hole circle (at -3.81 -1.27 270) (size 1.524 1.524) (drill 0.8128) (layers *.Cu *.Mask)
+    (pad "4" thru_hole circle (at -3.81 -1.27 90) (size 1.524 1.524) (drill 0.8128) (layers *.Cu *.Mask)
       (net 5 "/LED Row IO 1/ LDRow_Amps/Amp_OP_4") (pinfunction "CH3") (pintype "input"))
-    (pad "5" thru_hole circle (at -3.81 1.27 270) (size 1.524 1.524) (drill 0.8128) (layers *.Cu *.Mask)
+    (pad "5" thru_hole circle (at -3.81 1.27 90) (size 1.524 1.524) (drill 0.8128) (layers *.Cu *.Mask)
       (net 4 "/LED Row IO 1/ LDRow_Amps/Amp_OP_5") (pinfunction "CH4") (pintype "input"))
-    (pad "6" thru_hole circle (at -3.81 3.81 270) (size 1.524 1.524) (drill 0.8128) (layers *.Cu *.Mask)
+    (pad "6" thru_hole circle (at -3.81 3.81 90) (size 1.524 1.524) (drill 0.8128) (layers *.Cu *.Mask)
       (net 3 "/LED Row IO 1/ LDRow_Amps/Amp_OP_6") (pinfunction "CH5") (pintype "input"))
-    (pad "7" thru_hole circle (at -3.81 6.35 270) (size 1.524 1.524) (drill 0.8128) (layers *.Cu *.Mask)
+    (pad "7" thru_hole circle (at -3.81 6.35 90) (size 1.524 1.524) (drill 0.8128) (layers *.Cu *.Mask)
       (net 2 "/LED Row IO 1/ LDRow_Amps/Amp_OP_7") (pinfunction "CH6") (pintype "input"))
-    (pad "8" thru_hole circle (at -3.81 8.89 270) (size 1.524 1.524) (drill 0.8128) (layers *.Cu *.Mask)
+    (pad "8" thru_hole circle (at -3.81 8.89 90) (size 1.524 1.524) (drill 0.8128) (layers *.Cu *.Mask)
       (net 1 "/LED Row IO 1/ LDRow_Amps/Amp_OP_8") (pinfunction "CH7") (pintype "input"))
-    (pad "9" thru_hole circle (at 3.81 8.89 270) (size 1.524 1.524) (drill 0.8128) (layers *.Cu *.Mask)
+    (pad "9" thru_hole circle (at 3.81 8.89 90) (size 1.524 1.524) (drill 0.8128) (layers *.Cu *.Mask)
       (net 9 "GND") (pinfunction "DGND") (pintype "input"))
-    (pad "10" thru_hole circle (at 3.81 6.35 270) (size 1.524 1.524) (drill 0.8128) (layers *.Cu *.Mask)
+    (pad "10" thru_hole circle (at 3.81 6.35 90) (size 1.524 1.524) (drill 0.8128) (layers *.Cu *.Mask)
       (net 10 "/LED Row IO 1/ADC_SHDN") (pinfunction "SHDN/~{CS}") (pintype "input"))
-    (pad "11" thru_hole circle (at 3.81 3.81 270) (size 1.524 1.524) (drill 0.8128) (layers *.Cu *.Mask)
+    (pad "11" thru_hole circle (at 3.81 3.81 90) (size 1.524 1.524) (drill 0.8128) (layers *.Cu *.Mask)
       (net 11 "SPI_MOSI") (pinfunction "DIN") (pintype "input"))
-    (pad "12" thru_hole circle (at 3.81 1.27 270) (size 1.524 1.524) (drill 0.8128) (layers *.Cu *.Mask)
+    (pad "12" thru_hole circle (at 3.81 1.27 90) (size 1.524 1.524) (drill 0.8128) (layers *.Cu *.Mask)
       (net 12 "SPI_MISO_5V") (pinfunction "DOUT") (pintype "output"))
-    (pad "13" thru_hole circle (at 3.81 -1.27 270) (size 1.524 1.524) (drill 0.8128) (layers *.Cu *.Mask)
+    (pad "13" thru_hole circle (at 3.81 -1.27 90) (size 1.524 1.524) (drill 0.8128) (layers *.Cu *.Mask)
       (net 13 "SPI_SCK") (pinfunction "CLK") (pintype "input"))
-    (pad "14" thru_hole circle (at 3.81 -3.81 270) (size 1.524 1.524) (drill 0.8128) (layers *.Cu *.Mask)
+    (pad "14" thru_hole circle (at 3.81 -3.81 90) (size 1.524 1.524) (drill 0.8128) (layers *.Cu *.Mask)
       (net 9 "GND") (pinfunction "AGND") (pintype "power_in"))
-    (pad "15" thru_hole circle (at 3.81 -6.35 270) (size 1.524 1.524) (drill 0.8128) (layers *.Cu *.Mask)
+    (pad "15" thru_hole circle (at 3.81 -6.35 90) (size 1.524 1.524) (drill 0.8128) (layers *.Cu *.Mask)
       (net 14 "+5V") (pinfunction "VREF") (pintype "input"))
-    (pad "16" thru_hole circle (at 3.81 -8.89 270) (size 1.524 1.524) (drill 0.8128) (layers *.Cu *.Mask)
+    (pad "16" thru_hole circle (at 3.81 -8.89 90) (size 1.524 1.524) (drill 0.8128) (layers *.Cu *.Mask)
       (net 14 "+5V") (pinfunction "VDD") (pintype "power_in"))
   )
