File: hardware/8x8/8x8.kicad_pcb (KiCad board)
At the start: 2 copper layers, 408.6 x 315.4 mm, 250 parts

Commit message: Updated Footprints
Parts:
- Lvl_Sftr_1: value LSF0102DCH -> VSSOP8_SOT765-1_NEX
- SSR1: renamed from OC1; value CPC1125N -> TLP4176ATP_F; footprint Opto-coupler:footprints -> SSR:footprints
- SSR10: renamed from OC10; value CPC1125N -> TLP4176ATP_F; footprint Opto-coupler:footprints -> SSR:footprints
- SSR11: renamed from OC11; value CPC1125N -> TLP4176ATP_F; footprint Opto-coupler:footprints -> SSR:footprints
- SSR12: renamed from OC12; value CPC1125N -> TLP4176ATP_F; footprint Opto-coupler:footprints -> SSR:footprints
- SSR13: renamed from OC13; value CPC1125N -> TLP4176ATP_F; footprint Opto-coupler:footprints -> SSR:footprints
- SSR14: renamed from OC14; value CPC1125N -> TLP4176ATP_F; footprint Opto-coupler:footprints -> SSR:footprints
- SSR15: renamed from OC15; value CPC1125N -> TLP4176ATP_F; footprint Opto-coupler:footprints -> SSR:footprints
- SSR16: renamed from OC16; value CPC1125N -> TLP4176ATP_F; footprint Opto-coupler:footprints -> SSR:footprints
- SSR17: renamed from OC17; value CPC1125N -> TLP4176ATP_F; footprint Opto-coupler:footprints -> SSR:footprints
- SSR18: renamed from OC18; value CPC1125N -> TLP4176ATP_F; footprint Opto-coupler:footprints -> SSR:footprints
- SSR19: renamed from OC19; value CPC1125N -> TLP4176ATP_F; footprint Opto-coupler:footprints -> SSR:footprints
- SSR2: renamed from OC2; value CPC1125N -> TLP4176ATP_F; footprint Opto-coupler:footprints -> SSR:footprints
- SSR20: renamed from OC20; value CPC1125N -> TLP4176ATP_F; footprint Opto-coupler:footprints -> SSR:footprints
- SSR21: renamed from OC21; value CPC1125N -> TLP4176ATP_F; footprint Opto-coupler:footprints -> SSR:footprints
- SSR22: renamed from OC22; value CPC1125N -> TLP4176ATP_F; footprint Opto-coupler:footprints -> SSR:footprints
- SSR23: renamed from OC23; value CPC1125N -> TLP4176ATP_F; footprint Opto-coupler:footprints -> SSR:footprints
- SSR24: renamed from OC24; value CPC1125N -> TLP4176ATP_F; footprint Opto-coupler:footprints -> SSR:footprints
- SSR25: renamed from OC25; value CPC1125N -> TLP4176ATP_F; footprint Opto-coupler:footprints -> SSR:footprints
- SSR26: renamed from OC26; value CPC1125N -> TLP4176ATP_F; footprint Opto-coupler:footprints -> SSR:footprints
- SSR27: renamed from OC27; value CPC1125N -> TLP4176ATP_F; footprint Opto-coupler:footprints -> SSR:footprints
- SSR28: renamed from OC28; value CPC1125N -> TLP4176ATP_F; footprint Opto-coupler:footprints -> SSR:footprints
- SSR29: renamed from OC29; value CPC1125N -> TLP4176ATP_F; footprint Opto-coupler:footprints -> SSR:footprints
- SSR3: renamed from OC3; value CPC1125N -> TLP4176ATP_F; footprint Opto-coupler:footprints -> SSR:footprints
- SSR30: renamed from OC30; value CPC1125N -> TLP4176ATP_F; footprint Opto-coupler:footprints -> SSR:footprints
- SSR31: renamed from OC31; value CPC1125N -> TLP4176ATP_F; footprint Opto-coupler:footprints -> SSR:footprints
- SSR32: renamed from OC32; value CPC1125N -> TLP4176ATP_F; footprint Opto-coupler:footprints -> SSR:footprints
- SSR33: renamed from OC33; value CPC1125N -> TLP4176ATP_F; footprint Opto-coupler:footprints -> SSR:footprints
- SSR34: renamed from OC34; value CPC1125N -> TLP4176ATP_F; footprint Opto-coupler:footprints -> SSR:footprints
- SSR35: renamed from OC35; value CPC1125N -> TLP4176ATP_F; footprint Opto-coupler:footprints -> SSR:footprints
- SSR36: renamed from OC36; value CPC1125N -> TLP4176ATP_F; footprint Opto-coupler:footprints -> SSR:footprints
- SSR37: renamed from OC37; value CPC1125N -> TLP4176ATP_F; footprint Opto-coupler:footprints -> SSR:footprints
- SSR38: renamed from OC38; value CPC1125N -> TLP4176ATP_F; footprint Opto-coupler:footprints -> SSR:footprints
- SSR39: renamed from OC39; value CPC1125N -> TLP4176ATP_F; footprint Opto-coupler:footprints -> SSR:footprints
- SSR4: renamed from OC4; value CPC1125N -> TLP4176ATP_F; footprint Opto-coupler:footprints -> SSR:footprints
- SSR40: renamed from OC40; value CPC1125N -> TLP4176ATP_F; footprint Opto-coupler:footprints -> SSR:footprints
- SSR41: renamed from OC41; value CPC1125N -> TLP4176ATP_F; footprint Opto-coupler:footprints -> SSR:footprints
- SSR42: renamed from OC42; value CPC1125N -> TLP4176ATP_F; footprint Opto-coupler:footprints -> SSR:footprints
- SSR43: renamed from OC43; value CPC1125N -> TLP4176ATP_F; footprint Opto-coupler:footprints -> SSR:footprints
- SSR44: renamed from OC44; value CPC1125N -> TLP4176ATP_F; footprint Opto-coupler:footprints -> SSR:footprints
- SSR45: renamed from OC45; value CPC1125N -> TLP4176ATP_F; footprint Opto-coupler:footprints -> SSR:footprints
- SSR46: renamed from OC46; value CPC1125N -> TLP4176ATP_F; footprint Opto-coupler:footprints -> SSR:footprints
- SSR47: renamed from OC47; value CPC1125N -> TLP4176ATP_F; footprint Opto-coupler:footprints -> SSR:footprints
- SSR48: renamed from OC48; value CPC1125N -> TLP4176ATP_F; footprint Opto-coupler:footprints -> SSR:footprints
- SSR49: renamed from OC49; value CPC1125N -> TLP4176ATP_F; footprint Opto-coupler:footprints -> SSR:footprints
- SSR5: renamed from OC5; value CPC1125N -> TLP4176ATP_F; footprint Opto-coupler:footprints -> SSR:footprints
- SSR50: renamed from OC50; value CPC1125N -> TLP4176ATP_F; footprint Opto-coupler:footprints -> SSR:footprints
- SSR51: renamed from OC51; value CPC1125N -> TLP4176ATP_F; footprint Opto-coupler:footprints -> SSR:footprints
- SSR52: renamed from OC52; value CPC1125N -> TLP4176ATP_F; footprint Opto-coupler:footprints -> SSR:footprints
- SSR53: renamed from OC53; value CPC1125N -> TLP4176ATP_F; footprint Opto-coupler:footprints -> SSR:footprints
- SSR54: renamed from OC54; value CPC1125N -> TLP4176ATP_F; footprint Opto-coupler:footprints -> SSR:footprints
- SSR55: renamed from OC55; value CPC1125N -> TLP4176ATP_F; footprint Opto-coupler:footprints -> SSR:footprints
- SSR56: renamed from OC56; value CPC1125N -> TLP4176ATP_F; footprint Opto-coupler:footprints -> SSR:footprints
- SSR57: renamed from OC57; value CPC1125N -> TLP4176ATP_F; footprint Opto-coupler:footprints -> SSR:footprints
- SSR58: renamed from OC58; value CPC1125N -> TLP4176ATP_F; footprint Opto-coupler:footprints -> SSR:footprints
- SSR59: renamed from OC59; value CPC1125N -> TLP4176ATP_F; footprint Opto-coupler:footprints -> SSR:footprints
- SSR6: renamed from OC6; value CPC1125N -> TLP4176ATP_F; footprint Opto-coupler:footprints -> SSR:footprints
- SSR60: renamed from OC60; value CPC1125N -> TLP4176ATP_F; footprint Opto-coupler:footprints -> SSR:footprints
- SSR61: renamed from OC61; value CPC1125N -> TLP4176ATP_F; footprint Opto-coupler:footprints -> SSR:footprints
- SSR62: renamed from OC62; value CPC1125N -> TLP4176ATP_F; footprint Opto-coupler:footprints -> SSR:footprints
- SSR63: renamed from OC63; value CPC1125N -> TLP4176ATP_F; footprint Opto-coupler:footprints -> SSR:footprints
- SSR64: renamed from OC64; value CPC1125N -> TLP4176ATP_F; footprint Opto-coupler:footprints -> SSR:footprints
- SSR7: renamed from OC7; value CPC1125N -> TLP4176ATP_F; footprint Opto-coupler:footprints -> SSR:footprints
- SSR8: renamed from OC8; value CPC1125N -> TLP4176ATP_F; footprint Opto-coupler:footprints -> SSR:footprints
- SSR9: renamed from OC9; value CPC1125N -> TLP4176ATP_F; footprint Opto-coupler:footprints -> SSR:footprints

Commit message: Updated Footprints
Parts:
- removed ADC_1, ADC_2, ADC_3, ADC_4, ADC_5, ADC_6, ADC_7, ADC_8: MCP3008-I/P-DIP16, ADC:MCP3008-I&slash_P
- removed AMP_1, AMP_10, AMP_11, AMP_12, AMP_13, AMP_14, AMP_15, AMP_16, AMP_2, AMP_3, AMP_4, AMP_5, AMP_6, AMP_7, AMP_8, AMP_9: MCP619-I/SL, Op-Amp:footprints
- removed Addr_Sel_1, Addr_Sel_2, Addr_Sel_3, Addr_Sel_4, Addr_Sel_5, Addr_Sel_6: 100K, Resistor_THT:R_Axial_DIN0207_L6.3mm_D2.5mm_P7.62mm_Horizontal
- removed Amp_Fdbk_1, Amp_Fdbk_10, Amp_Fdbk_11, Amp_Fdbk_12, Amp_Fdbk_13, Amp_Fdbk_14, Amp_Fdbk_15, Amp_Fdbk_16, Amp_Fdbk_17, Amp_Fdbk_18, Amp_Fdbk_19, Amp_Fdbk_2, Amp_Fdbk_20, Amp_Fdbk_21, Amp_Fdbk_22, Amp_Fdbk_23, Amp_Fdbk_24, Amp_Fdbk_25, Amp_Fdbk_26, Amp_Fdbk_27, Amp_Fdbk_28, Amp_Fdbk_29, Amp_Fdbk_3, Amp_Fdbk_30, Amp_Fdbk_31, Amp_Fdbk_32, Amp_Fdbk_33, Amp_Fdbk_34, Amp_Fdbk_35, Amp_Fdbk_36, Amp_Fdbk_37, Amp_Fdbk_38, Amp_Fdbk_39, Amp_Fdbk_4, Amp_Fdbk_40, Amp_Fdbk_41, Amp_Fdbk_42, Amp_Fdbk_43, Amp_Fdbk_44, Amp_Fdbk_45, Amp_Fdbk_46, Amp_Fdbk_47, Amp_Fdbk_48, Amp_Fdbk_49, Amp_Fdbk_5, Amp_Fdbk_50, Amp_Fdbk_51, Amp_Fdbk_52, Amp_Fdbk_53, Amp_Fdbk_54, Amp_Fdbk_55, Amp_Fdbk_56, Amp_Fdbk_57, Amp_Fdbk_58, Amp_Fdbk_59, Amp_Fdbk_6, Amp_Fdbk_60, Amp_Fdbk_61, Amp_Fdbk_62, Amp_Fdbk_63, Amp_Fdbk_64, Amp_Fdbk_7, Amp_Fdbk_8, Amp_Fdbk_9: 2M, Resistor_THT:R_Axial_DIN0207_L6.3mm_D2.5mm_P7.62mm_Horizontal
- removed DEMUX_1: 74HC138D-Q100,118, DEMUX:footprints
- removed Drv_I_Sel_1, Drv_I_Sel_2, Drv_I_Sel_3, Drv_I_Sel_4, Drv_I_Sel_5, Drv_I_Sel_6, Drv_I_Sel_7, Drv_I_Sel_8: 2K, Resistor_THT:R_Axial_DIN0207_L6.3mm_D2.5mm_P7.62mm_Horizontal
- removed Drv_RST_PU_1, Drv_RST_PU_2, Drv_RST_PU_3, Drv_RST_PU_4, Drv_RST_PU_5, Drv_RST_PU_6, Drv_RST_PU_7, Drv_RST_PU_8: 10K, Resistor_THT:R_Axial_DIN0207_L6.3mm_D2.5mm_P7.62mm_Horizontal
- removed LED_Driver_1, LED_Driver_2, LED_Driver_3, LED_Driver_4, LED_Driver_5, LED_Driver_6, LED_Driver_7, LED_Driver_8: PCA9956BTWY, LED Driver:SOP50P640X110-39N
- removed Lvl_Sftr_1: VSSOP8_SOT765-1_NEX, Level Shifter:LSF0102DCH
- removed Pin_Header_1: Conn_02x16_Odd_Even, Connector_PinHeader_2.54mm:PinHeader_2x16_P2.54mm_Vertical
- removed Rev_Bias_Sel_1: 100K, Potentiometer_THT:Potentiometer_Runtron_RM-065_Vertical
- removed SSR1, SSR10, SSR11, SSR12, SSR13, SSR14, SSR15, SSR16, SSR17, SSR18, SSR19, SSR2, SSR20, SSR21, SSR22, SSR23, SSR24, SSR25, SSR26, SSR27, SSR28, SSR29, SSR3, SSR30, SSR31, SSR32, SSR33, SSR34, SSR35, SSR36, SSR37, SSR38, SSR39, SSR4, SSR40, SSR41, SSR42, SSR43, SSR44, SSR45, SSR46, SSR47, SSR48, SSR49, SSR5, SSR50, SSR51, SSR52, SSR53, SSR54, SSR55, SSR56, SSR57, SSR58, SSR59, SSR6, SSR60, SSR61, SSR62, SSR63, SSR64, SSR7, SSR8, SSR9: TLP4176ATP_F, SSR:footprints
- added AD1: MCP3008-I/P-DIP16, ADC:MCP3008-I&slash_P, B.Cu at (157.0, 12.0)
- added AD2: MCP3008-I/P-DIP16, ADC:MCP3008-I&slash_P, F.Cu at (147.3, 92.7)
- added AD3: MCP3008-I/P-DIP16, ADC:MCP3008-I&slash_P, F.Cu at (176.5, 114.6)
- added AD4: MCP3008-I/P-DIP16, ADC:MCP3008-I&slash_P, F.Cu at (268.2, 61.5)
- added AD5: MCP3008-I/P-DIP16, ADC:MCP3008-I&slash_P, F.Cu at (223.4, 16.8)
- added AD6: MCP3008-I/P-DIP16, ADC:MCP3008-I&slash_P, F.Cu at (223.4, 61.5)
- added AD7: MCP3008-I/P-DIP16, ADC:MCP3008-I&slash_P, F.Cu at (313.0, 16.8)
- added AD8: MCP3008-I/P-DIP16, ADC:MCP3008-I&slash_P, F.Cu at (268.2, 16.8)
- added ADSEL1: 100K, Resistor TH:footprints, F.Cu at (176.6, 48.3)
- added ADSEL2: 100K, Resistor TH:footprints, B.Cu at (85.7, 55.4)
- added ADSEL3: 100K, Resistor TH:footprints, B.Cu at (82.6, 55.4)
- added ADSEL4: 100K, Resistor TH:footprints, F.Cu at (183.8, 16.7)
- added ADSEL5: 100K, Resistor TH:footprints, F.Cu at (205.3, 5.57)
- added ADSEL6: 100K, Resistor TH:footprints, F.Cu at (205.3, 9.62)
- added AMP1: MCP619-I/SL, Op-Amp:footprints, F.Cu at (152.9, 1.27)
- added AMP10: MCP619-I/SL, Op-Amp:footprints, F.Cu at (342.5, 106.2)
- added AMP11: MCP619-I/SL, Op-Amp:footprints, F.Cu at (366.8, 53.4)
- added AMP12: MCP619-I/SL, Op-Amp:footprints, F.Cu at (356.0, 61.5)
- added AMP13: MCP619-I/SL, Op-Amp:footprints, F.Cu at (333.4, 53.4)
- added AMP14: MCP619-I/SL, Op-Amp:footprints, F.Cu at (322.6, 61.5)
- added AMP15: MCP619-I/SL, Op-Amp:footprints, F.Cu at (319.9, 98.1)
- added AMP16: MCP619-I/SL, Op-Amp:footprints, F.Cu at (309.9, 106.7)
- added AMP2: MCP619-I/SL, Op-Amp:footprints, F.Cu at (161.5, 1.27)
- added AMP3: MCP619-I/SL, Op-Amp:footprints, F.Cu at (378.2, 8.65)
- added AMP4: MCP619-I/SL, Op-Amp:footprints, F.Cu at (367.4, 16.7)
- added AMP5: MCP619-I/SL, Op-Amp:footprints, F.Cu at (400.2, 53.4)
- added AMP6: MCP619-I/SL, Op-Amp:footprints, F.Cu at (389.4, 61.5)
- added AMP7: MCP619-I/SL, Op-Amp:footprints, F.Cu at (411.6, 8.65)
- added AMP8: MCP619-I/SL, Op-Amp:footprints, F.Cu at (400.8, 16.7)
- added AMP9: MCP619-I/SL, Op-Amp:footprints, F.Cu at (353.3, 98.1)
- added DMX1: 74HC138D-Q100,118, DEMUX:footprints, F.Cu at (182.3, 9.13)
- added DRV1: PCA9956BTWY, LED Driver:SOP50P640X110-39N, F.Cu at (10.2, 55.4)
- added DRV2: PCA9956BTWY, LED Driver:SOP50P640X110-39N, B.Cu at (93.8, 55.4)
- added DRV3: PCA9956BTWY, LED Driver:SOP50P640X110-39N, F.Cu at (175.6, 132.1)
- added DRV4: PCA9956BTWY, LED Driver:SOP50P640X110-39N, F.Cu at (267.2, 79.0)
- added DRV5: PCA9956BTWY, LED Driver:SOP50P640X110-39N, F.Cu at (222.4, 34.2)
- added DRV6: PCA9956BTWY, LED Driver:SOP50P640X110-39N, F.Cu at (222.4, 79.0)
- added DRV7: PCA9956BTWY, LED Driver:SOP50P640X110-39N, F.Cu at (312.1, 34.2)
- added DRV8: PCA9956BTWY, LED Driver:SOP50P640X110-39N, F.Cu at (267.2, 34.2)
- added FDB1: 2M, Resistor TH:footprints, F.Cu at (146.8, 1.27)
- added FDB10: 2M, Resistor TH:footprints, F.Cu at (357.9, 5.57)
- added FDB11: 2M, Resistor TH:footprints, F.Cu at (357.9, 25.8)
- added FDB12: 2M, Resistor TH:footprints, F.Cu at (357.9, 17.7)
- added FDB13: 2M, Resistor TH:footprints, F.Cu at (357.9, 13.7)
- added FDB14: 2M, Resistor TH:footprints, F.Cu at (368.7, 5.57)
- added FDB15: 2M, Resistor TH:footprints, F.Cu at (357.9, 9.62)
- added FDB16: 2M, Resistor TH:footprints, F.Cu at (357.9, 21.8)
- added FDB17: 2M, Resistor TH:footprints, F.Cu at (390.6, 54.4)
- added FDB18: 2M, Resistor TH:footprints, F.Cu at (379.8, 50.3)
- added FDB19: 2M, Resistor TH:footprints, F.Cu at (379.8, 70.6)
- added FDB2: 2M, Resistor TH:footprints, F.Cu at (149.0, 25.0)
- added FDB20: 2M, Resistor TH:footprints, F.Cu at (379.8, 62.5)
- added FDB21: 2M, Resistor TH:footprints, F.Cu at (379.8, 58.4)
- added FDB22: 2M, Resistor TH:footprints, F.Cu at (390.6, 50.3)
- added FDB23: 2M, Resistor TH:footprints, F.Cu at (379.8, 54.4)
- added FDB24: 2M, Resistor TH:footprints, F.Cu at (379.8, 66.5)
- added FDB25: 2M, Resistor TH:footprints, F.Cu at (402.0, 9.62)
- added FDB26: 2M, Resistor TH:footprints, F.Cu at (391.3, 5.57)
- added FDB27: 2M, Resistor TH:footprints, F.Cu at (391.3, 25.8)
- added FDB28: 2M, Resistor TH:footprints, F.Cu at (391.3, 17.7)
- added FDB29: 2M, Resistor TH:footprints, F.Cu at (391.3, 13.7)
- added FDB3: 2M, Resistor TH:footprints, F.Cu at (138.0, 28.0)
- added FDB30: 2M, Resistor TH:footprints, F.Cu at (402.0, 5.57)
- added FDB31: 2M, Resistor TH:footprints, F.Cu at (391.3, 9.62)
- added FDB32: 2M, Resistor TH:footprints, F.Cu at (391.3, 21.8)
- added FDB33: 2M, Resistor TH:footprints, F.Cu at (343.7, 99.1)
- added FDB34: 2M, Resistor TH:footprints, F.Cu at (333.0, 95.1)
- added FDB35: 2M, Resistor TH:footprints, F.Cu at (333.0, 115.3)
- added FDB36: 2M, Resistor TH:footprints, F.Cu at (333.0, 107.2)
- added FDB37: 2M, Resistor TH:footprints, F.Cu at (333.0, 103.2)
- added FDB38: 2M, Resistor TH:footprints, F.Cu at (343.7, 95.1)
- added FDB39: 2M, Resistor TH:footprints, F.Cu at (333.0, 99.1)
- added FDB4: 2M, Resistor TH:footprints, F.Cu at (138.0, 6.00)
- added FDB40: 2M, Resistor TH:footprints, F.Cu at (333.0, 111.3)
- added FDB41: 2M, Resistor TH:footprints, F.Cu at (357.2, 54.4)
- added FDB42: 2M, Resistor TH:footprints, F.Cu at (346.4, 50.3)
- added FDB43: 2M, Resistor TH:footprints, F.Cu at (346.4, 70.6)
- added FDB44: 2M, Resistor TH:footprints, F.Cu at (346.4, 62.5)
- added FDB45: 2M, Resistor TH:footprints, F.Cu at (346.4, 58.4)
- added FDB46: 2M, Resistor TH:footprints, F.Cu at (357.2, 50.3)
- added FDB47: 2M, Resistor TH:footprints, F.Cu at (346.4, 54.4)
- added FDB48: 2M, Resistor TH:footprints, F.Cu at (346.4, 66.5)
- added FDB49: 2M, Resistor TH:footprints, F.Cu at (323.8, 54.4)
- added FDB5: 2M, Resistor TH:footprints, F.Cu at (127.0, 11.0)
- added FDB50: 2M, Resistor TH:footprints, F.Cu at (313.1, 50.3)
- added FDB51: 2M, Resistor TH:footprints, F.Cu at (313.1, 70.6)
- added FDB52: 2M, Resistor TH:footprints, F.Cu at (313.1, 62.5)
- added FDB53: 2M, Resistor TH:footprints, F.Cu at (313.1, 58.4)
- added FDB54: 2M, Resistor TH:footprints, F.Cu at (323.8, 50.3)
- added FDB55: 2M, Resistor TH:footprints, F.Cu at (313.1, 54.4)
- added FDB56: 2M, Resistor TH:footprints, F.Cu at (313.1, 66.5)
- added FDB57: 2M, Resistor TH:footprints, F.Cu at (310.4, 99.1)
- added FDB58: 2M, Resistor TH:footprints, F.Cu at (299.6, 95.1)
- added FDB59: 2M, Resistor TH:footprints, F.Cu at (299.6, 115.3)
- added FDB6: 2M, Resistor TH:footprints, F.Cu at (117.0, 22.0)
- added FDB60: 2M, Resistor TH:footprints, F.Cu at (299.6, 107.2)
- added FDB61: 2M, Resistor TH:footprints, F.Cu at (299.6, 103.2)
- added FDB62: 2M, Resistor TH:footprints, F.Cu at (310.4, 95.1)
- added FDB63: 2M, Resistor TH:footprints, F.Cu at (299.6, 99.1)
- added FDB64: 2M, Resistor TH:footprints, F.Cu at (299.6, 111.3)
- added FDB7: 2M, Resistor TH:footprints, F.Cu at (127.0, 28.0)
- added FDB8: 2M, Resistor TH:footprints, F.Cu at (117.0, 17.0)
- added FDB9: 2M, Resistor TH:footprints, F.Cu at (368.7, 9.62)
- added ISEL1: 2K, Resistor TH:footprints, F.Cu at (176.5, 54.6)
- added ISEL2: 2K, Resistor TH:footprints, B.Cu at (93.8, 48.3)
- added ISEL3: 2K, Resistor TH:footprints, F.Cu at (187.3, 103.4)
- added ISEL4: 2K, Resistor TH:footprints, F.Cu at (278.9, 50.3)
- added ISEL5: 2K, Resistor TH:footprints, F.Cu at (234.1, 5.57)
- added ISEL6: 2K, Resistor TH:footprints, F.Cu at (234.1, 50.3)
- added ISEL7: 2K, Resistor TH:footprints, F.Cu at (323.8, 5.57)
- added ISEL8: 2K, Resistor TH:footprints, F.Cu at (278.9, 5.57)
- added PH1: Conn_02x16_Odd_Even, Connector_PinHeader_2.54mm:PinHeader_2x16_P2.54mm_Vertical, F.Cu at (472.4, 57.1)
- added PU1: 10K, Resistor TH:footprints, F.Cu at (176.6, 95.0)
- added PU2: 10K, Resistor TH:footprints, B.Cu at (93.8, 62.5)
- added PU3: 10K, Resistor TH:footprints, F.Cu at (176.6, 139.8)
- added PU4: 10K, Resistor TH:footprints, F.Cu at (268.2, 86.7)
- added PU5: 10K, Resistor TH:footprints, F.Cu at (223.4, 41.9)
- added PU6: 10K, Resistor TH:footprints, F.Cu at (223.4, 86.7)
- added PU7: 10K, Resistor TH:footprints, F.Cu at (313.1, 41.9)
- added PU8: 10K, Resistor TH:footprints, F.Cu at (268.2, 41.9)
- added RBSEL1: 100K, Potentiometer_THT:Potentiometer_Runtron_RM-065_Vertical, F.Cu at (190.7, 13.7)
- added SFTR1: LSF0102DCH, Level Shifter:LSF0102DCH, F.Cu at (200.0, 14.3)
- added SR1: TLP4176ATP_F, SSR:footprints, F.Cu at (111.8, -21.3)
- added SR10: TLP4176ATP_F, SSR:footprints, F.Cu at (133.2, 81.1)
- added SR11: TLP4176ATP_F, SSR:footprints, F.Cu at (142.4, 77.1)
- added SR12: TLP4176ATP_F, SSR:footprints, F.Cu at (151.7, 77.1)
- added SR13: TLP4176ATP_F, SSR:footprints, F.Cu at (143.9, 70.0)
- added SR14: TLP4176ATP_F, SSR:footprints, F.Cu at (131.2, 94.7)
- added SR15: TLP4176ATP_F, SSR:footprints, F.Cu at (153.2, 70.0)
- added SR16: TLP4176ATP_F, SSR:footprints, F.Cu at (133.2, 74.0)
- added SR17: TLP4176ATP_F, SSR:footprints, F.Cu at (195.8, 120.1)
- added SR18: TLP4176ATP_F, SSR:footprints, F.Cu at (186.5, 117.0)
- added SR19: TLP4176ATP_F, SSR:footprints, F.Cu at (195.8, 113.0)
- added SR2: TLP4176ATP_F, SSR:footprints, F.Cu at (111.6, -16.3)
- added SR20: TLP4176ATP_F, SSR:footprints, F.Cu at (205.0, 113.0)
- added SR21: TLP4176ATP_F, SSR:footprints, F.Cu at (197.3, 105.8)
- added SR22: TLP4176ATP_F, SSR:footprints, F.Cu at (184.6, 130.6)
- added SR23: TLP4176ATP_F, SSR:footprints, F.Cu at (206.5, 105.8)
- added SR24: TLP4176ATP_F, SSR:footprints, F.Cu at (186.5, 109.9)
- added SR25: TLP4176ATP_F, SSR:footprints, F.Cu at (287.5, 67.0)
- added SR26: TLP4176ATP_F, SSR:footprints, F.Cu at (278.2, 63.9)
- added SR27: TLP4176ATP_F, SSR:footprints, F.Cu at (287.5, 59.9)
- added SR28: TLP4176ATP_F, SSR:footprints, F.Cu at (296.7, 59.9)
- added SR29: TLP4176ATP_F, SSR:footprints, F.Cu at (289.0, 52.7)
- added SR3: TLP4176ATP_F, SSR:footprints, F.Cu at (111.8, -10.8)
- added SR30: TLP4176ATP_F, SSR:footprints, F.Cu at (276.3, 77.5)
- added SR31: TLP4176ATP_F, SSR:footprints, F.Cu at (298.2, 52.7)
- added SR32: TLP4176ATP_F, SSR:footprints, F.Cu at (278.2, 56.8)
- added SR33: TLP4176ATP_F, SSR:footprints, F.Cu at (242.6, 22.2)
- added SR34: TLP4176ATP_F, SSR:footprints, F.Cu at (233.4, 19.2)
- added SR35: TLP4176ATP_F, SSR:footprints, F.Cu at (242.6, 15.1)
- added SR36: TLP4176ATP_F, SSR:footprints, F.Cu at (251.9, 15.1)
- added SR37: TLP4176ATP_F, SSR:footprints, F.Cu at (244.1, 7.96)
- added SR38: TLP4176ATP_F, SSR:footprints, F.Cu at (231.4, 32.7)
- added SR39: TLP4176ATP_F, SSR:footprints, F.Cu at (253.4, 7.96)
- added SR4: TLP4176ATP_F, SSR:footprints, F.Cu at (111.8, -5.59)
- added SR40: TLP4176ATP_F, SSR:footprints, F.Cu at (233.4, 12.0)
- added SR41: TLP4176ATP_F, SSR:footprints, F.Cu at (242.6, 67.0)
- added SR42: TLP4176ATP_F, SSR:footprints, F.Cu at (233.4, 63.9)
- added SR43: TLP4176ATP_F, SSR:footprints, F.Cu at (242.6, 59.9)
- added SR44: TLP4176ATP_F, SSR:footprints, F.Cu at (251.9, 59.9)
- added SR45: TLP4176ATP_F, SSR:footprints, F.Cu at (244.1, 52.7)
- added SR46: TLP4176ATP_F, SSR:footprints, F.Cu at (231.4, 77.5)
- added SR47: TLP4176ATP_F, SSR:footprints, F.Cu at (253.4, 52.7)
- added SR48: TLP4176ATP_F, SSR:footprints, F.Cu at (233.4, 56.8)
- added SR49: TLP4176ATP_F, SSR:footprints, F.Cu at (332.3, 22.2)
- added SR5: TLP4176ATP_F, SSR:footprints, F.Cu at (94.0, 73.0)
- added SR50: TLP4176ATP_F, SSR:footprints, F.Cu at (323.0, 19.2)
- added SR51: TLP4176ATP_F, SSR:footprints, F.Cu at (332.3, 15.1)
- added SR52: TLP4176ATP_F, SSR:footprints, F.Cu at (341.5, 15.1)
- added SR53: TLP4176ATP_F, SSR:footprints, F.Cu at (333.8, 7.96)
- added SR54: TLP4176ATP_F, SSR:footprints, F.Cu at (321.1, 32.7)
- added SR55: TLP4176ATP_F, SSR:footprints, F.Cu at (343.0, 7.96)
- added SR56: TLP4176ATP_F, SSR:footprints, F.Cu at (323.0, 12.0)
- added SR57: TLP4176ATP_F, SSR:footprints, F.Cu at (287.5, 22.2)
- added SR58: TLP4176ATP_F, SSR:footprints, F.Cu at (278.2, 19.2)
- added SR59: TLP4176ATP_F, SSR:footprints, F.Cu at (287.5, 15.1)
- added SR6: TLP4176ATP_F, SSR:footprints, F.Cu at (184.6, 85.8)
- added SR60: TLP4176ATP_F, SSR:footprints, F.Cu at (296.7, 15.1)
- added SR61: TLP4176ATP_F, SSR:footprints, F.Cu at (289.0, 7.96)
- added SR62: TLP4176ATP_F, SSR:footprints, F.Cu at (276.3, 32.7)
- added SR63: TLP4176ATP_F, SSR:footprints, F.Cu at (298.2, 7.96)
- added SR64: TLP4176ATP_F, SSR:footprints, F.Cu at (278.2, 12.0)
- added SR7: TLP4176ATP_F, SSR:footprints, F.Cu at (107.7, 56.6)
- added SR8: TLP4176ATP_F, SSR:footprints, F.Cu at (114.0, 72.0)
- added SR9: TLP4176ATP_F, SSR:footprints, F.Cu at (142.4, 84.2)
- moved LD5 38.9 mm to (21.3, 59.4)
- moved LD6 38.9 mm to (29.0, 59.4)
- moved LD8 38.9 mm to (44.2, 59.4)
- moved LD7 38.9 mm to (36.6, 59.4)
- moved LD12 35.9 mm to (74.6, 51.8)
- moved LD10 35.9 mm to (59.4, 51.8)
- moved LD11 35.9 mm to (67.0, 51.8)
- moved LD9 35.9 mm to (51.8, 51.8)
- moved LD13 20.4 mm to (51.8, 59.4)
- moved LD14 20.4 mm to (59.4, 59.4)
- moved LD15 20.4 mm to (67.0, 59.4)
- moved LD16 20.4 mm to (74.6, 59.4)
- moved LD1 20.4 mm to (21.3, 51.8)
- moved LD2 20.4 mm to (29.0, 51.8)
- moved LD3 20.4 mm to (36.6, 51.8)
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
Commit message: Completed Major Routing
Parts:
- AD2, AD3, AD4, AD5, AD6, AD7, AD8, DMX1, DRV1, DRV3, DRV4, DRV5, DRV6, DRV7, DRV8, FDB1, FDB10, FDB11, FDB12, FDB13, FDB14, FDB15, FDB16, FDB17, FDB18, FDB19, FDB2, FDB20, FDB21, FDB22, FDB23, FDB24, FDB25, FDB26, FDB27, FDB28, FDB29, FDB3, FDB30, FDB31, FDB32, FDB33, FDB34, FDB35, FDB36, FDB37, FDB38, FDB39, FDB4, FDB40, FDB41, FDB42, FDB43, FDB44, FDB45, FDB46, FDB47, FDB48, FDB49, FDB5, FDB50, FDB51, FDB52, FDB53, FDB54, FDB55, FDB56, FDB57, FDB58, FDB59, FDB6, FDB60, FDB61, FDB62, FDB63, FDB64, FDB7, FDB8, FDB9, PH1, RBSEL1, SFTR1, SR1, SR10, SR11, SR12, SR13, SR14, SR15, SR16, SR17, SR18, SR19, SR2, SR20, SR21, SR22, SR23, SR24, SR25, SR26, SR27, SR28, SR29, SR3, SR30, SR31, SR32, SR33, SR34, SR35, SR36, SR37, SR38, SR39, SR4, SR40, SR41, SR42, SR43, SR44, SR45, SR46, SR47, SR48, SR49, SR5, SR50, SR51, SR52, SR53, SR54, SR55, SR56, SR57, SR58, SR59, SR6, SR60, SR61, SR62, SR63, SR64, SR7, SR8, SR9: moved to B.Cu
- ADSEL2, ADSEL3, ISEL2, PU2: moved to F.Cu
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Connections:
- net /LED Row IO 1/ADC_SHDN renamed /LED 4x2 Left 1/ADC_SHDN
- net /LED Row IO 1/Drv_AD0 renamed /LED 4x2 Left 1/Drv_AD0
- net /LED Row IO 1/Drv_AD1 renamed /LED 4x2 Left 1/Drv_AD1
- net /LED Row IO 1/LDRow/LD1_R renamed /LED 4x2 Left 1/LD1_R
- net /LED Row IO 1/LDRow/LD2_R renamed /LED 4x2 Left 1/LD2_R
- net /LED Row IO 1/LDRow/LD3_R renamed /LED 4x2 Left 1/LD3_R
- net /LED Row IO 1/LDRow/LD4_R renamed /LED 4x2 Left 1/LD4_R
- net /LED Row IO 1/LDRow/LD5_G renamed /LED 4x2 Left 1/LD5_G
- net /LED Row IO 1/LDRow/LD5_R renamed /LED 4x2 Left 1/LD5_R
- net /LED Row IO 1/LDRow/LD6_R renamed /LED 4x2 Left 1/LD6_R
- net /LED Row IO 1/LDRow/LD7_R renamed /LED 4x2 Left 1/LD7_R
- net /LED Row IO 1/LDRow/LD8_R renamed /LED 4x2 Left 1/LD8_R
- net /LED Row IO 2/ADC_SHDN renamed /LED 4x2 Right 1/ADC_SHDN
- net /LED Row IO 2/Drv_AD0 renamed /LED 4x2 Right 1/Drv_AD0
- net /LED Row IO 2/Drv_AD1 renamed /LED 4x2 Right 1/Drv_AD1
- net /LED Row IO 2/LDRow/LD1_R renamed /LED 4x2 Right 1/LD1_R
- net /LED Row IO 2/LDRow/LD2_B renamed /LED 4x2 Right 1/LD2_B
- net /LED Row IO 2/LDRow/LD2_G renamed /LED 4x2 Right 1/LD2_G
- net /LED Row IO 2/LDRow/LD2_R renamed /LED 4x2 Right 1/LD2_R
- net /LED Row IO 2/LDRow/LD3_R renamed /LED 4x2 Right 1/LD3_R
- net /LED Row IO 2/LDRow/LD4_R renamed /LED 4x2 Right 1/LD4_R
- net /LED Row IO 2/LDRow/LD5_R renamed /LED 4x2 Right 1/LD5_R
- net /LED Row IO 2/LDRow/LD6_R renamed /LED 4x2 Right 1/LD6_R
- net /LED Row IO 2/LDRow/LD7_B renamed /LED 4x2 Right 1/LD7_B
- net /LED Row IO 2/LDRow/LD7_R renamed /LED 4x2 Right 1/LD7_R
- net /LED Row IO 2/LDRow/LD8_R renamed /LED 4x2 Right 1/LD8_R
- net /LED Row IO 3/ADC_SHDN renamed /LED 4x2 Left 2/ADC_SHDN
- net /LED Row IO 3/Drv_AD1 renamed /LED 4x2 Left 2/Drv_AD1
- net /LED Row IO 3/LDRow/LD1_R renamed /LED 4x2 Left 2/LD1_R
- net /LED Row IO 3/LDRow/LD2_R renamed /LED 4x2 Left 2/LD2_R
- net /LED Row IO 3/LDRow/LD3_R renamed /LED 4x2 Left 2/LD3_R
- net /LED Row IO 3/LDRow/LD4_R renamed /LED 4x2 Left 2/LD4_R
- net /LED Row IO 3/LDRow/LD5_G renamed /LED 4x2 Left 2/LD5_G
- net /LED Row IO 3/LDRow/LD5_R renamed /LED 4x2 Left 2/LD5_R
- net /LED Row IO 3/LDRow/LD6_R renamed /LED 4x2 Left 2/LD6_R
- net /LED Row IO 3/LDRow/LD7_R renamed /LED 4x2 Left 2/LD7_R
- net /LED Row IO 3/LDRow/LD8_R renamed /LED 4x2 Left 2/LD8_R
- net /LED Row IO 4/ADC_SHDN renamed /LED 4x2 Right 2/ADC_SHDN
- net /LED Row IO 4/Drv_AD1 renamed /LED 4x2 Right 2/Drv_AD1
- net /LED Row IO 4/LDRow/LD1_R renamed /LED 4x2 Right 2/LD1_R
- net /LED Row IO 4/LDRow/LD2_B renamed /LED 4x2 Right 2/LD2_B
- net /LED Row IO 4/LDRow/LD2_G renamed /LED 4x2 Right 2/LD2_G
- net /LED Row IO 4/LDRow/LD2_R renamed /LED 4x2 Right 2/LD2_R
- net /LED Row IO 4/LDRow/LD3_R renamed /LED 4x2 Right 2/LD3_R
- net /LED Row IO 4/LDRow/LD4_R renamed /LED 4x2 Right 2/LD4_R
- net /LED Row IO 4/LDRow/LD5_R renamed /LED 4x2 Right 2/LD5_R
- net /LED Row IO 4/LDRow/LD6_R renamed /LED 4x2 Right 2/LD6_R
- net /LED Row IO 4/LDRow/LD7_B renamed /LED 4x2 Right 2/LD7_B
- net /LED Row IO 4/LDRow/LD7_R renamed /LED 4x2 Right 2/LD7_R
- net /LED Row IO 4/LDRow/LD8_R renamed /LED 4x2 Right 2/LD8_R
- net /LED Row IO 5/ADC_SHDN renamed /LED 4x2 Left 3/ADC_SHDN
- net /LED Row IO 5/Drv_AD0 renamed /LED 4x2 Left 3/Drv_AD0
- net /LED Row IO 5/Drv_AD1 renamed /LED 4x2 Left 3/Drv_AD1
- net /LED Row IO 5/LDRow/LD1_R renamed /LED 4x2 Left 3/LD1_R
- net /LED Row IO 5/LDRow/LD2_R renamed /LED 4x2 Left 3/LD2_R
- net /LED Row IO 5/LDRow/LD3_R renamed /LED 4x2 Left 3/LD3_R
- net /LED Row IO 5/LDRow/LD4_R renamed /LED 4x2 Left 3/LD4_R
- net /LED Row IO 5/LDRow/LD5_G renamed /LED 4x2 Left 3/LD5_G
- net /LED Row IO 5/LDRow/LD5_R renamed /LED 4x2 Left 3/LD5_R
- net /LED Row IO 5/LDRow/LD6_R renamed /LED 4x2 Left 3/LD6_R
- net /LED Row IO 5/LDRow/LD7_R renamed /LED 4x2 Left 3/LD7_R
- net /LED Row IO 5/LDRow/LD8_R renamed /LED 4x2 Left 3/LD8_R
- net /LED Row IO 6/ADC_SHDN renamed /LED 4x2 Right 3/ADC_SHDN
- net /LED Row IO 6/Drv_AD0 renamed /LED 4x2 Right 3/Drv_AD0
- net /LED Row IO 6/Drv_AD1 renamed /LED 4x2 Right 3/Drv_AD1
- net /LED Row IO 6/LDRow/LD1_R renamed /LED 4x2 Right 3/LD1_R
- net /LED Row IO 6/LDRow/LD2_B renamed /LED 4x2 Right 3/LD2_B
- net /LED Row IO 6/LDRow/LD2_G renamed /LED 4x2 Right 3/LD2_G
- net /LED Row IO 6/LDRow/LD2_R renamed /LED 4x2 Right 3/LD2_R
- net /LED Row IO 6/LDRow/LD3_R renamed /LED 4x2 Right 3/LD3_R
- net /LED Row IO 6/LDRow/LD4_R renamed /LED 4x2 Right 3/LD4_R
- net /LED Row IO 6/LDRow/LD5_R renamed /LED 4x2 Right 3/LD5_R
- net /LED Row IO 6/LDRow/LD6_R renamed /LED 4x2 Right 3/LD6_R
- net /LED Row IO 6/LDRow/LD7_B renamed /LED 4x2 Right 3/LD7_B
- net /LED Row IO 6/LDRow/LD7_R renamed /LED 4x2 Right 3/LD7_R
- net /LED Row IO 6/LDRow/LD8_R renamed /LED 4x2 Right 3/LD8_R
- net /LED Row IO 7/ADC_SHDN renamed /LED 4x2 Left 4/ADC_SHDN
- net /LED Row IO 7/Drv_AD0 renamed /LED 4x2 Left 4/Drv_AD0
- net /LED Row IO 7/Drv_AD1 renamed /LED 4x2 Left 4/Drv_AD1
- net /LED Row IO 7/LDRow/LD1_R renamed /LED 4x2 Left 4/LD1_R
- net /LED Row IO 7/LDRow/LD2_R renamed /LED 4x2 Left 4/LD2_R
- net /LED Row IO 7/LDRow/LD3_R renamed /LED 4x2 Left 4/LD3_R
- net /LED Row IO 7/LDRow/LD4_R renamed /LED 4x2 Left 4/LD4_R
- net /LED Row IO 7/LDRow/LD5_G renamed /LED 4x2 Left 4/LD5_G
- net /LED Row IO 7/LDRow/LD5_R renamed /LED 4x2 Left 4/LD5_R
- net /LED Row IO 7/LDRow/LD6_R renamed /LED 4x2 Left 4/LD6_R
- net /LED Row IO 7/LDRow/LD7_R renamed /LED 4x2 Left 4/LD7_R
- net /LED Row IO 7/LDRow/LD8_R renamed /LED 4x2 Left 4/LD8_R
- net /LED Row IO 8/ADC_SHDN renamed /LED 4x2 Right 4/ADC_SHDN
- net /LED Row IO 8/Drv_AD1 renamed /LED 4x2 Right 4/Drv_AD1
- net /LED Row IO 8/LDRow/LD1_R renamed /LED 4x2 Right 4/LD1_R
- net /LED Row IO 8/LDRow/LD2_B renamed /LED 4x2 Right 4/LD2_B
- net /LED Row IO 8/LDRow/LD2_G renamed /LED 4x2 Right 4/LD2_G
- net /LED Row IO 8/LDRow/LD2_R renamed /LED 4x2 Right 4/LD2_R
- net /LED Row IO 8/LDRow/LD3_R renamed /LED 4x2 Right 4/LD3_R
- net /LED Row IO 8/LDRow/LD4_R renamed /LED 4x2 Right 4/LD4_R
- net /LED Row IO 8/LDRow/LD5_R renamed /LED 4x2 Right 4/LD5_R
- net /LED Row IO 8/LDRow/LD6_R renamed /LED 4x2 Right 4/LD6_R
- net /LED Row IO 8/LDRow/LD7_B renamed /LED 4x2 Right 4/LD7_B
- net /LED Row IO 8/LDRow/LD7_R renamed /LED 4x2 Right 4/LD7_R
- net /LED Row IO 8/LDRow/LD8_R renamed /LED 4x2 Right 4/LD8_R
- net Net-(DRV1-Pad6) renamed /LED 4x2 Left 1/SR1_R
- net Net-(DRV3-Pad6) renamed /LED 4x2 Left 2/SR1_R
- net Net-(DRV5-Pad6) renamed /LED 4x2 Left 3/SR1_R
- net Net-(DRV7-Pad6) renamed /LED 4x2 Left 4/SR1_R
- AD1 pad 1: /LED Row IO 1/ LDRow_Amps/Amp_OP_1 -> /LED 4x2 Left 1/ LDRow_Amps1/Amp_OP_6
- AD1 pad 2: /LED Row IO 1/ LDRow_Amps/Amp_OP_2 -> /LED 4x2 Left 1/ LDRow_Amps1/Amp_OP_5
- AD1 pad 3: /LED Row IO 1/ LDRow_Amps/Amp_OP_3 -> /LED 4x2 Left 1/ LDRow_Amps1/Amp_OP_2
- AD1 pad 4: /LED Row IO 1/ LDRow_Amps/Amp_OP_4 -> /LED 4x2 Left 1/ LDRow_Amps1/Amp_OP_1
- AD1 pad 5: /LED Row IO 1/ LDRow_Amps/Amp_OP_5 -> /LED 4x2 Left 1/ LDRow_Amps1/Amp_OP_4
- AD1 pad 6: /LED Row IO 1/ LDRow_Amps/Amp_OP_6 -> /LED 4x2 Left 1/ LDRow_Amps1/Amp_OP_3
- AD1 pad 7: /LED Row IO 1/ LDRow_Amps/Amp_OP_7 -> /LED 4x2 Left 1/ LDRow_Amps1/Amp_OP_8
- AD1 pad 8: /LED Row IO 1/ LDRow_Amps/Amp_OP_8 -> /LED 4x2 Left 1/ LDRow_Amps1/Amp_OP_7
- AD2 pad 1: /LED Row IO 2/ LDRow_Amps/Amp_OP_1 -> /LED 4x2 Right 1/ LDRow_Amps/Amp_OP_4
- AD2 pad 2: /LED Row IO 2/ LDRow_Amps/Amp_OP_2 -> /LED 4x2 Right 1/ LDRow_Amps/Amp_OP_3
- AD2 pad 3: /LED Row IO 2/ LDRow_Amps/Amp_OP_3 -> /LED 4x2 Right 1/ LDRow_Amps/Amp_OP_8
- AD2 pad 4: /LED Row IO 2/ LDRow_Amps/Amp_OP_4 -> /LED 4x2 Right 1/ LDRow_Amps/Amp_OP_7
- AD2 pad 5: /LED Row IO 2/ LDRow_Amps/Amp_OP_5 -> /LED 4x2 Right 1/ LDRow_Amps/Amp_OP_6
- AD2 pad 6: /LED Row IO 2/ LDRow_Amps/Amp_OP_6 -> /LED 4x2 Right 1/ LDRow_Amps/Amp_OP_5
- AD2 pad 7: /LED Row IO 2/ LDRow_Amps/Amp_OP_7 -> /LED 4x2 Right 1/ LDRow_Amps/Amp_OP_2
- AD2 pad 8: /LED Row IO 2/ LDRow_Amps/Amp_OP_8 -> /LED 4x2 Right 1/ LDRow_Amps/Amp_OP_1
- AD3 pad 1: /LED Row IO 3/ LDRow_Amps/Amp_OP_1 -> /LED 4x2 Left 2/ LDRow_Amps1/Amp_OP_6
- AD3 pad 2: /LED Row IO 3/ LDRow_Amps/Amp_OP_2 -> /LED 4x2 Left 2/ LDRow_Amps1/Amp_OP_5
- AD3 pad 3: /LED Row IO 3/ LDRow_Amps/Amp_OP_3 -> /LED 4x2 Left 2/ LDRow_Amps1/Amp_OP_2
- AD3 pad 4: /LED Row IO 3/ LDRow_Amps/Amp_OP_4 -> /LED 4x2 Left 2/ LDRow_Amps1/Amp_OP_1
- AD3 pad 5: /LED Row IO 3/ LDRow_Amps/Amp_OP_5 -> /LED 4x2 Left 2/ LDRow_Amps1/Amp_OP_4
- AD3 pad 6: /LED Row IO 3/ LDRow_Amps/Amp_OP_6 -> /LED 4x2 Left 2/ LDRow_Amps1/Amp_OP_3
- AD3 pad 7: /LED Row IO 3/ LDRow_Amps/Amp_OP_7 -> /LED 4x2 Left 2/ LDRow_Amps1/Amp_OP_8
- AD3 pad 8: /LED Row IO 3/ LDRow_Amps/Amp_OP_8 -> /LED 4x2 Left 2/ LDRow_Amps1/Amp_OP_7
- AD4 pad 1: /LED Row IO 4/ LDRow_Amps/Amp_OP_1 -> /LED 4x2 Right 2/ LDRow_Amps/Amp_OP_4
- AD4 pad 2: /LED Row IO 4/ LDRow_Amps/Amp_OP_2 -> /LED 4x2 Right 2/ LDRow_Amps/Amp_OP_3
- AD4 pad 3: /LED Row IO 4/ LDRow_Amps/Amp_OP_3 -> /LED 4x2 Right 2/ LDRow_Amps/Amp_OP_8
- AD4 pad 4: /LED Row IO 4/ LDRow_Amps/Amp_OP_4 -> /LED 4x2 Right 2/ LDRow_Amps/Amp_OP_7
- AD4 pad 5: /LED Row IO 4/ LDRow_Amps/Amp_OP_5 -> /LED 4x2 Right 2/ LDRow_Amps/Amp_OP_6
- AD4 pad 6: /LED Row IO 4/ LDRow_Amps/Amp_OP_6 -> /LED 4x2 Right 2/ LDRow_Amps/Amp_OP_5
- AD4 pad 7: /LED Row IO 4/ LDRow_Amps/Amp_OP_7 -> /LED 4x2 Right 2/ LDRow_Amps/Amp_OP_2
- AD4 pad 8: /LED Row IO 4/ LDRow_Amps/Amp_OP_8 -> /LED 4x2 Right 2/ LDRow_Amps/Amp_OP_1
- AD5 pad 1: /LED Row IO 5/ LDRow_Amps/Amp_OP_1 -> /LED 4x2 Left 3/ LDRow_Amps1/Amp_OP_6
- AD5 pad 2: /LED Row IO 5/ LDRow_Amps/Amp_OP_2 -> /LED 4x2 Left 3/ LDRow_Amps1/Amp_OP_5
- AD5 pad 3: /LED Row IO 5/ LDRow_Amps/Amp_OP_3 -> /LED 4x2 Left 3/ LDRow_Amps1/Amp_OP_2
- AD5 pad 4: /LED Row IO 5/ LDRow_Amps/Amp_OP_4 -> /LED 4x2 Left 3/ LDRow_Amps1/Amp_OP_1
- AD5 pad 5: /LED Row IO 5/ LDRow_Amps/Amp_OP_5 -> /LED 4x2 Left 3/ LDRow_Amps1/Amp_OP_4
- AD5 pad 6: /LED Row IO 5/ LDRow_Amps/Amp_OP_6 -> /LED 4x2 Left 3/ LDRow_Amps1/Amp_OP_3
- AD5 pad 7: /LED Row IO 5/ LDRow_Amps/Amp_OP_7 -> /LED 4x2 Left 3/ LDRow_Amps1/Amp_OP_8
- AD5 pad 8: /LED Row IO 5/ LDRow_Amps/Amp_OP_8 -> /LED 4x2 Left 3/ LDRow_Amps1/Amp_OP_7
- AD6 pad 1: /LED Row IO 6/ LDRow_Amps/Amp_OP_1 -> /LED 4x2 Right 3/ LDRow_Amps/Amp_OP_4
- AD6 pad 2: /LED Row IO 6/ LDRow_Amps/Amp_OP_2 -> /LED 4x2 Right 3/ LDRow_Amps/Amp_OP_3
- AD6 pad 3: /LED Row IO 6/ LDRow_Amps/Amp_OP_3 -> /LED 4x2 Right 3/ LDRow_Amps/Amp_OP_8
- AD6 pad 4: /LED Row IO 6/ LDRow_Amps/Amp_OP_4 -> /LED 4x2 Right 3/ LDRow_Amps/Amp_OP_7
- AD6 pad 5: /LED Row IO 6/ LDRow_Amps/Amp_OP_5 -> /LED 4x2 Right 3/ LDRow_Amps/Amp_OP_6
- AD6 pad 6: /LED Row IO 6/ LDRow_Amps/Amp_OP_6 -> /LED 4x2 Right 3/ LDRow_Amps/Amp_OP_5
- AD6 pad 7: /LED Row IO 6/ LDRow_Amps/Amp_OP_7 -> /LED 4x2 Right 3/ LDRow_Amps/Amp_OP_2
- AD6 pad 8: /LED Row IO 6/ LDRow_Amps/Amp_OP_8 -> /LED 4x2 Right 3/ LDRow_Amps/Amp_OP_1
- AD7 pad 1: /LED Row IO 7/ LDRow_Amps/Amp_OP_1 -> /LED 4x2 Left 4/ LDRow_Amps1/Amp_OP_6
- AD7 pad 2: /LED Row IO 7/ LDRow_Amps/Amp_OP_2 -> /LED 4x2 Left 4/ LDRow_Amps1/Amp_OP_5
- AD7 pad 3: /LED Row IO 7/ LDRow_Amps/Amp_OP_3 -> /LED 4x2 Left 4/ LDRow_Amps1/Amp_OP_2
- AD7 pad 4: /LED Row IO 7/ LDRow_Amps/Amp_OP_4 -> /LED 4x2 Left 4/ LDRow_Amps1/Amp_OP_1
- AD7 pad 5: /LED Row IO 7/ LDRow_Amps/Amp_OP_5 -> /LED 4x2 Left 4/ LDRow_Amps1/Amp_OP_4
- AD7 pad 6: /LED Row IO 7/ LDRow_Amps/Amp_OP_6 -> /LED 4x2 Left 4/ LDRow_Amps1/Amp_OP_3
- AD7 pad 7: /LED Row IO 7/ LDRow_Amps/Amp_OP_7 -> /LED 4x2 Left 4/ LDRow_Amps1/Amp_OP_8
- AD7 pad 8: /LED Row IO 7/ LDRow_Amps/Amp_OP_8 -> /LED 4x2 Left 4/ LDRow_Amps1/Amp_OP_7
- AD8 pad 1: /LED Row IO 8/ LDRow_Amps/Amp_OP_1 -> /LED 4x2 Right 4/ LDRow_Amps/Amp_OP_4
- AD8 pad 2: /LED Row IO 8/ LDRow_Amps/Amp_OP_2 -> /LED 4x2 Right 4/ LDRow_Amps/Amp_OP_3
- AD8 pad 3: /LED Row IO 8/ LDRow_Amps/Amp_OP_3 -> /LED 4x2 Right 4/ LDRow_Amps/Amp_OP_8
- AD8 pad 4: /LED Row IO 8/ LDRow_Amps/Amp_OP_4 -> /LED 4x2 Right 4/ LDRow_Amps/Amp_OP_7
- AD8 pad 5: /LED Row IO 8/ LDRow_Amps/Amp_OP_5 -> /LED 4x2 Right 4/ LDRow_Amps/Amp_OP_6
- AD8 pad 6: /LED Row IO 8/ LDRow_Amps/Amp_OP_6 -> /LED 4x2 Right 4/ LDRow_Amps/Amp_OP_5
- AD8 pad 7: /LED Row IO 8/ LDRow_Amps/Amp_OP_7 -> /LED 4x2 Right 4/ LDRow_Amps/Amp_OP_2
- AD8 pad 8: /LED Row IO 8/ LDRow_Amps/Amp_OP_8 -> /LED 4x2 Right 4/ LDRow_Amps/Amp_OP_1
- AMP1 pad 1: /LED Row IO 1/ LDRow_Amps/Amp_OP_1 -> /LED 4x2 Left 1/ LDRow_Amps1/Amp_OP_1
- AMP1 pad 13: /LED Row IO 1/ LDRow_Amps/Amp_IP_4 -> /LED 4x2 Left 1/ LDRow_Amps1/Amp_IP_4
- AMP1 pad 14: /LED Row IO 1/ LDRow_Amps/Amp_OP_4 -> /LED 4x2 Left 1/ LDRow_Amps1/Amp_OP_4
- AMP1 pad 2: /LED Row IO 1/ LDRow_Amps/Amp_IP_1 -> /LED 4x2 Left 1/ LDRow_Amps1/Amp_IP_1
- AMP1 pad 6: /LED Row IO 1/ LDRow_Amps/Amp_IP_2 -> /LED 4x2 Left 1/ LDRow_Amps1/Amp_IP_2
- AMP1 pad 7: /LED Row IO 1/ LDRow_Amps/Amp_OP_2 -> /LED 4x2 Left 1/ LDRow_Amps1/Amp_OP_2
- AMP1 pad 8: /LED Row IO 1/ LDRow_Amps/Amp_OP_3 -> /LED 4x2 Left 1/ LDRow_Amps1/Amp_OP_3
- AMP1 pad 9: /LED Row IO 1/ LDRow_Amps/Amp_IP_3 -> /LED 4x2 Left 1/ LDRow_Amps1/Amp_IP_3
- AMP10 pad 1: /LED Row IO 5/ LDRow_Amps/Amp_OP_5 -> /LED 4x2 Left 3/ LDRow_Amps1/Amp_OP_5
- AMP10 pad 13: /LED Row IO 5/ LDRow_Amps/Amp_IP_8 -> /LED 4x2 Left 3/ LDRow_Amps1/Amp_IP_8
- AMP10 pad 14: /LED Row IO 5/ LDRow_Amps/Amp_OP_8 -> /LED 4x2 Left 3/ LDRow_Amps1/Amp_OP_8
- AMP10 pad 2: /LED Row IO 5/ LDRow_Amps/Amp_IP_5 -> /LED 4x2 Left 3/ LDRow_Amps1/Amp_IP_5
- AMP10 pad 6: /LED Row IO 5/ LDRow_Amps/Amp_IP_6 -> /LED 4x2 Left 3/ LDRow_Amps1/Amp_IP_6
- AMP10 pad 7: /LED Row IO 5/ LDRow_Amps/Amp_OP_6 -> /LED 4x2 Left 3/ LDRow_Amps1/Amp_OP_6
- AMP10 pad 8: /LED Row IO 5/ LDRow_Amps/Amp_OP_7 -> /LED 4x2 Left 3/ LDRow_Amps1/Amp_OP_7
- AMP10 pad 9: /LED Row IO 5/ LDRow_Amps/Amp_IP_7 -> /LED 4x2 Left 3/ LDRow_Amps1/Amp_IP_7
- AMP11 pad 1: /LED Row IO 6/ LDRow_Amps/Amp_OP_1 -> /LED 4x2 Right 3/ LDRow_Amps/Amp_OP_1
- AMP11 pad 13: /LED Row IO 6/ LDRow_Amps/Amp_IP_4 -> /LED 4x2 Right 3/ LDRow_Amps/Amp_IP_4
- AMP11 pad 14: /LED Row IO 6/ LDRow_Amps/Amp_OP_4 -> /LED 4x2 Right 3/ LDRow_Amps/Amp_OP_4
- AMP11 pad 2: /LED Row IO 6/ LDRow_Amps/Amp_IP_1 -> /LED 4x2 Right 3/ LDRow_Amps/Amp_IP_1
- AMP11 pad 6: /LED Row IO 6/ LDRow_Amps/Amp_IP_2 -> /LED 4x2 Right 3/ LDRow_Amps/Amp_IP_2
- AMP11 pad 7: /LED Row IO 6/ LDRow_Amps/Amp_OP_2 -> /LED 4x2 Right 3/ LDRow_Amps/Amp_OP_2
- AMP11 pad 8: /LED Row IO 6/ LDRow_Amps/Amp_OP_3 -> /LED 4x2 Right 3/ LDRow_Amps/Amp_OP_3
- AMP11 pad 9: /LED Row IO 6/ LDRow_Amps/Amp_IP_3 -> /LED 4x2 Right 3/ LDRow_Amps/Amp_IP_3
- AMP12 pad 1: /LED Row IO 6/ LDRow_Amps/Amp_OP_5 -> /LED 4x2 Right 3/ LDRow_Amps/Amp_OP_5
- AMP12 pad 13: /LED Row IO 6/ LDRow_Amps/Amp_IP_8 -> /LED 4x2 Right 3/ LDRow_Amps/Amp_IP_8
- AMP12 pad 14: /LED Row IO 6/ LDRow_Amps/Amp_OP_8 -> /LED 4x2 Right 3/ LDRow_Amps/Amp_OP_8
- AMP12 pad 2: /LED Row IO 6/ LDRow_Amps/Amp_IP_5 -> /LED 4x2 Right 3/ LDRow_Amps/Amp_IP_5
- AMP12 pad 6: /LED Row IO 6/ LDRow_Amps/Amp_IP_6 -> /LED 4x2 Right 3/ LDRow_Amps/Amp_IP_6
- AMP12 pad 7: /LED Row IO 6/ LDRow_Amps/Amp_OP_6 -> /LED 4x2 Right 3/ LDRow_Amps/Amp_OP_6
- AMP12 pad 8: /LED Row IO 6/ LDRow_Amps/Amp_OP_7 -> /LED 4x2 Right 3/ LDRow_Amps/Amp_OP_7
- AMP12 pad 9: /LED Row IO 6/ LDRow_Amps/Amp_IP_7 -> /LED 4x2 Right 3/ LDRow_Amps/Amp_IP_7
- AMP13 pad 1: /LED Row IO 7/ LDRow_Amps/Amp_OP_1 -> /LED 4x2 Left 4/ LDRow_Amps1/Amp_OP_1
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Routing:
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Other:
- board size 408.6 x 315.4 mm -> 321.8 x 10.2 mm

Commit message: Completed 8x8 Routing
Parts:
- SFTR1: value LSF0102DCH -> VSSOP8_SOT765-1_NEX
- moved SFTR1 94.2 mm to (94.7, -192.4), turned to -90 degrees
- moved PH1 89.9 mm to (137.3, -191.1)
- moved DMX1 61.0 mm to (146.7, -192.2)
- moved RBSEL1 40.5 mm to (224.2, -195.4), turned to 180 degrees
Connections:
- DMX1 pad 10: /LED 4x2 Right 3/ADC_SHDN -> /LED 4x2 Right 1/ADC_SHDN
- DMX1 pad 11: /LED 4x2 Left 3/ADC_SHDN -> /LED 4x2 Right 3/ADC_SHDN
- DMX1 pad 12: /LED 4x2 Right 2/ADC_SHDN -> /LED 4x2 Left 4/ADC_SHDN
- DMX1 pad 14: /LED 4x2 Right 1/ADC_SHDN -> /LED 4x2 Left 3/ADC_SHDN
- DMX1 pad 7: /LED 4x2 Right 4/ADC_SHDN -> /LED 4x2 Right 2/ADC_SHDN
- DMX1 pad 9: /LED 4x2 Left 4/ADC_SHDN -> /LED 4x2 Right 4/ADC_SHDN
Routing:
- net GND: track 483.8 -> 1186.0 mm, vias 8 -> 16
- net SPI_MISO_5V: track 86.3 -> 612.2 mm, vias 0 -> 4
- net SPI_MOSI: track 81.2 -> 605.6 mm, vias 0 -> 4
- net SPI_SCK: track 91.4 -> 610.0 mm, vias 0 -> 2
- net +5V: track 1512.3 -> 1752.0 mm, vias 1 -> 8
- net I2C_SCL: track 0.00 -> 235.6 mm, vias 0 -> 15
- net I2C_SDA_5V: track 0.00 -> 232.1 mm, vias 0 -> 15
- net /LED 4x2 Right 4/ADC_SHDN: track 0.00 -> 197.4 mm
- net RB Voltage: track 758.9 -> 954.7 mm, vias 24 -> 34
- net /LED 4x2 Left 4/ADC_SHDN: track 0.00 -> 193.7 mm
- net /LED 4x2 Left 3/ADC_SHDN: track 0.00 -> 183.2 mm
- net /LED 4x2 Right 3/ADC_SHDN: track 0.00 -> 175.4 mm
- net /LED 4x2 Right 2/ADC_SHDN: track 0.00 -> 170.6 mm
- net /LED 4x2 Left 2/ADC_SHDN: track 0.00 -> 162.9 mm
- net /LED 4x2 Left 1/ADC_SHDN: track 0.00 -> 158.5 mm
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Other:
- board size 321.8 x 10.2 mm -> 322.6 x 80 mm
