File: hardware/8x8/8x8.kicad_pcb (KiCad board)
At the start: 2 copper layers, 322.6 x 80 mm, 250 parts

Commit message: Updated PCB
Routing:
- added copper zone on B.Cu, net GND
- added copper zone on F.Cu, net GND
