File: hardware/8x8/8x8.kicad_pcb (KiCad board)
At the start: 2 copper layers, 322.6 x 80 mm, 250 parts

Commit message: Updated One 4x2-Right Block
Parts:
- moved AD6 8.59 mm to (279.9, -150.4)
- moved ADSEL4 4.51 mm to (104.0, -165.8)
- moved AMP5 4.51 mm to (77.9, -165.8)
- moved AMP6 4.51 mm to (40.9, -165.8)
- moved DRV3 4.51 mm to (111.2, -165.8)
- moved FDB17 4.51 mm to (91.4, -168.9)
- moved FDB18 4.51 mm to (64.3, -168.9)
- moved FDB19 4.51 mm to (64.3, -162.8)
- moved FDB20 4.51 mm to (91.4, -162.8)
- moved FDB21 4.51 mm to (54.5, -168.9)
- moved FDB22 4.51 mm to (27.3, -168.8)
- moved FDB23 4.51 mm to (27.3, -162.7)
- moved FDB24 4.51 mm to (54.5, -162.8)
- moved ISEL3 4.51 mm to (100.9, -165.8)
- moved PU3 4.51 mm to (97.9, -165.8)
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Routing:
- net +5V: track 1752.0 -> 714.5 mm, vias 8 -> 4
- net GND: track 1186.0 -> 676.4 mm, vias 16 -> 9
- net RB Voltage: track 954.7 -> 540.0 mm, vias 34 -> 14
- net +9V: track 1003.9 -> 644.0 mm, vias 8 -> 3
- net I2C_SCL: track 235.6 -> 78.3 mm, vias 15 -> 7
- net I2C_SDA_5V: track 232.1 -> 77.3 mm, vias 15 -> 7
- net /LED 4x2 Right 2/LD5_R: track 121.0 -> 0.00 mm, vias 2 -> 0
- net /LED 4x2 Right 1/LD5_R: track 121.0 -> 0.00 mm, vias 2 -> 0
- net /LED 4x2 Right 4/LD5_R: track 121.0 -> 0.00 mm, vias 2 -> 0
- net /LED 4x2 Right 4/LD1_R: track 120.9 -> 0.00 mm, vias 2 -> 0
- net /LED 4x2 Right 2/LD1_R: track 120.9 -> 0.00 mm, vias 2 -> 0
- net /LED 4x2 Right 1/LD1_R: track 120.9 -> 0.00 mm, vias 2 -> 0
- net /LED 4x2 Left 2/LD4_R: track 115.0 -> 0.00 mm, vias 2 -> 0
- net /LED 4x2 Left 2/LD8_R: track 114.7 -> 0.00 mm, vias 2 -> 0
- net /LED 4x2 Right 2/LD6_R: track 104.1 -> 0.00 mm, vias 2 -> 0
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- removed copper zone on B.Cu, net GND
- removed copper zone on F.Cu, net GND

Commit message: Updated All Right Blocks & One 4x2 Left Block
Parts:
- moved AD8 10.2 mm to (290.1, -135.2)
- moved AD4 10.1 mm to (290.1, -165.7)
- moved AD3 9.12 mm to (16.9, -165.7)
- moved AD2 8.59 mm to (279.9, -180.9)
- moved ADSEL3 7.22 mm to (184.6, -181.0)
- moved FDB28 4.17 mm to (269.4, -162.6)
- moved AMP16 4.17 mm to (218.8, -135.2)
- moved AMP4 4.17 mm to (218.8, -180.9)
- moved AMP7 4.17 mm to (255.8, -165.8)
- moved DRV2 4.17 mm to (195.0, -181.0)
- moved FDB10 4.17 mm to (242.3, -184.0)
- moved FDB11 4.17 mm to (242.3, -177.8)
- moved FDB14 4.17 mm to (205.2, -184.1)
- moved FDB15 4.17 mm to (205.2, -177.9)
- moved FDB29 4.17 mm to (232.5, -168.8)
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Routing:
- net GND: track 676.4 -> 237.2 mm, vias 9 -> 3
- net SPI_SCK: track 519.9 -> 117.2 mm
- net SPI_MOSI: track 516.0 -> 114.4 mm, vias 2 -> 0
- net SPI_MISO_5V: track 522.4 -> 121.5 mm, vias 2 -> 0
- net +9V: track 644.0 -> 370.2 mm, vias 3 -> 0
- net /LED 4x2 Left 4/ADC_SHDN: track 193.7 -> 0.00 mm
- net /LED 4x2 Left 3/ADC_SHDN: track 183.2 -> 0.00 mm
- net /LED 4x2 Left 2/ADC_SHDN: track 162.9 -> 0.00 mm
- net /LED 4x2 Right 1/ADC_SHDN: track 142.0 -> 0.00 mm
- net /LED 4x2 Right 3/ADC_SHDN: track 140.6 -> 0.00 mm
- net /LED 4x2 Right 2/ADC_SHDN: track 135.6 -> 0.00 mm
- net /LED 4x2 Right 4/ADC_SHDN: track 132.3 -> 0.00 mm
- net /LED 4x2 Right 4/LD5_R: track 0.00 -> 122.8 mm, vias 0 -> 2
- net /LED 4x2 Right 4/LD1_R: track 0.00 -> 117.3 mm, vias 0 -> 2
- net /LED 4x2 Right 2/LD1_R: track 0.00 -> 117.3 mm, vias 0 -> 2
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
Commit message: Completed Block Routing. Communication Left
Parts:
- moved AD1 11.9 mm to (6.99, -181.0)
- moved AD5 11.9 mm to (7.01, -150.5)
- moved AD7 9.12 mm to (16.9, -135.2)
- moved ISEL1 4.52 mm to (100.9, -181.0)
- moved AMP9 4.51 mm to (77.9, -150.5)
- moved FDB2 4.51 mm to (64.2, -184.1)
- moved FDB3 4.51 mm to (64.2, -178.0)
- moved FDB50 4.51 mm to (64.2, -138.4)
- moved FDB51 4.51 mm to (64.2, -132.3)
- moved FDB38 4.51 mm to (27.3, -153.6)
- moved FDB39 4.51 mm to (27.3, -147.5)
- moved SR52 4.51 mm to (36.3, -138.3)
- moved SR56 4.51 mm to (36.3, -132.2)
- moved AMP1 4.51 mm to (77.8, -181.1)
- moved AMP10 4.51 mm to (40.9, -150.5)
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Routing:
- net RB Voltage: track 632.9 -> 1332.5 mm
- net +5V: track 697.5 -> 1387.5 mm, vias 6 -> 9
- net +9V: track 370.2 -> 966.1 mm, vias 0 -> 5
- net GND: track 237.2 -> 455.5 mm, vias 3 -> 9
- net I2C_SCL: track 80.6 -> 226.0 mm, vias 5 -> 8
- net I2C_SDA_5V: track 85.3 -> 229.1 mm, vias 5 -> 8
- net /LED 4x2 Left 1/ADC_SHDN: track 132.3 -> 0.00 mm
- net /LED 4x2 Left 4/LD8_R: track 0.00 -> 104.5 mm, vias 0 -> 2
- net /LED 4x2 Left 1/LD8_R: track 0.00 -> 104.5 mm, vias 0 -> 2
- net /LED 4x2 Left 3/LD8_R: track 0.00 -> 104.5 mm, vias 0 -> 2
- net /LED 4x2 Left 3/LD4_R: track 0.00 -> 104.2 mm, vias 0 -> 2
- net /LED 4x2 Left 4/LD4_R: track 0.00 -> 104.2 mm, vias 0 -> 2
- net /LED 4x2 Left 1/LD4_R: track 0.00 -> 104.2 mm, vias 0 -> 2
- net /LED 4x2 Left 1/LD3_R: track 0.00 -> 93.6 mm, vias 0 -> 2
- net /LED 4x2 Left 4/LD3_R: track 0.00 -> 93.6 mm, vias 0 -> 2
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