File: hardware/electronics/PCB/2x2/2x2.kicad_pcb (KiCad board)
At the start: 2 copper layers, 54.5 x 23.2 mm, 21 parts

Commit message: Added Screen Antenna Skeleton
Parts:
- SFTR1: value VSSOP8_SOT765-1_NEX -> LSF0102DCH
